File: ergodonk_pcb/ergodonk_pcb.kicad_sch (KiCad schematic)
At the start: 120 parts, among them J1 AudioJack4, Q1 TIP120

Commit message: Created Cherry MX Doublesided mini-e footprint variant and updated schematic
Parts:
- removed SW? (x2): SW_PUSH_LED, SofleRGB:Choc_Hotswap_SK6812MiniE, symbol SofleKeyboard:SW_PUSH_LED
- added SW, SW? (x47): SW_PUSH_LED, SofleRGB:Choc_Hotswap_SK6812MiniE, symbol SofleKeyboard:SW_PUSH_LED
- SWLH1, SWLH11, SWLH12, SWLH13, SWLH14, SWLH15, SWLH16, SWLH17, SWLH18, SWLH2, SWLH22, SWLH23, SWLH24, SWLH25, SWLH26, SWLH27, SWLH28, SWLH3, SWLH32, SWLH33, SWLH34, SWLH35, SWLH36, SWLH37, SWLH38, SWLH4, SWLH42, SWLH43, SWLH44, SWLH45, SWLH46, SWLH48, SWLH5, SWLH52, SWLH53, SWLH54, SWLH58, SWLH6, SWLH7, SWLH8: value SW_PUSH -> SW_PUSH_LED; footprint ergodonk_kicad_library:CherryMX_Hotswap -> SofleRGB:Choc_Hotswap_SK6812MiniE; symbol kbd:SW_PUSH -> SofleKeyboard:SW_PUSH_LED
- SWLH21: value SW_PUSH -> SW_PUSH_LED; footprint ergodonk_kicad_library:CherryMX_Hotswap_1.5u -> SofleRGB:Choc_Hotswap_SK6812MiniE; symbol kbd:SW_PUSH -> SofleKeyboard:SW_PUSH_LED
- SWLH31: value SW_PUSH -> SW_PUSH_LED; footprint ergodonk_kicad_library:CherryMX_Hotswap_1.75u_ergodonk -> SofleRGB:Choc_Hotswap_SK6812MiniE; symbol kbd:SW_PUSH -> SofleKeyboard:SW_PUSH_LED
- SWLH41, SWLH56, SWLH57: value SW_PUSH -> SW_PUSH_LED; footprint ergodonk_kicad_library:CherryMX_Hotswap_2u_ergodonk_Stabs -> SofleRGB:Choc_Hotswap_SK6812MiniE; symbol kbd:SW_PUSH -> SofleKeyboard:SW_PUSH_LED
- SWLH50, SWLH51: value SW_PUSH -> SW_PUSH_LED; footprint ergodonk_kicad_library:CherryMX_Hotswap_1.25u_ergodonk -> SofleRGB:Choc_Hotswap_SK6812MiniE; symbol kbd:SW_PUSH -> SofleKeyboard:SW_PUSH_LED
- SWLH55: value SW_PUSH -> SW_PUSH_LED; footprint ergodonk_kicad_library:CherryMX_Hotswap_1.25u_Vert_ergodonk -> SofleRGB:Choc_Hotswap_SK6812MiniE; symbol kbd:SW_PUSH -> SofleKeyboard:SW_PUSH_LED
Connections:
- net GND: now also SW.3 (GND), SW?.3 (GND), SW?.3 (GND), SW?.3 (GND), SW?.3 (GND), SW?.3 (GND), SW?.3 (GND), SW?.3 (GND), SW?.3 (GND), SW?.3 (GND), SW?.3 (GND), SW?.3 (GND), SW?.3 (GND), SW?.3 (GND), SW?.3 (GND), SW?.3 (GND), SW?.3 (GND), SW?.3 (GND), SW?.3 (GND), SW?.3 (GND), SW?.3 (GND), SW?.3 (GND), SW?.3 (GND), SW?.3 (GND), SW?.3 (GND), SW?.3 (GND), SW?.3 (GND), SW?.3 (GND), SW?.3 (GND), SW?.3 (GND), SW?.3 (GND), SW?.3 (GND), SW?.3 (GND), SW?.3 (GND), SW?.3 (GND), SW?.3 (GND), SW?.3 (GND), SW?.3 (GND), SW?.3 (GND), SW?.3 (GND), SW?.3 (GND), SW?.3 (GND), SW?.3 (GND), SW?.3 (GND), SW?.3 (GND), SW?.3 (GND), SW?.3 (GND), SW?.3 (GND)
- net SW47A: now also SWLH17.6, SWLH27.6, SWLH37.6, SWLH57.6, SWLH7.6; no longer SWLH17.1, SWLH27.1, SWLH37.1, SWLH57.1, SWLH7.1
- net VDD: now also SW.1 (VDD), SW?.1 (VDD), SW?.1 (VDD), SW?.1 (VDD), SW?.1 (VDD), SW?.1 (VDD), SW?.1 (VDD), SW?.1 (VDD), SW?.1 (VDD), SW?.1 (VDD), SW?.1 (VDD), SW?.1 (VDD), SW?.1 (VDD), SW?.1 (VDD), SW?.1 (VDD), SW?.1 (VDD), SW?.1 (VDD), SW?.1 (VDD), SW?.1 (VDD), SW?.1 (VDD), SW?.1 (VDD), SW?.1 (VDD), SW?.1 (VDD), SW?.1 (VDD), SW?.1 (VDD), SW?.1 (VDD), SW?.1 (VDD), SW?.1 (VDD), SW?.1 (VDD), SW?.1 (VDD), SW?.1 (VDD), SW?.1 (VDD), SW?.1 (VDD), SW?.1 (VDD), SW?.1 (VDD), SW?.1 (VDD), SW?.1 (VDD), SW?.1 (VDD), SW?.1 (VDD), SW?.1 (VDD), SW?.1 (VDD), SW?.1 (VDD), SW?.1 (VDD), SW?.1 (VDD), SW?.1 (VDD), SW?.1 (VDD), SW?.1 (VDD), SW?.1 (VDD)
- net col0: now also SWLH50.6; no longer SWLH50.1
- net col1: now also SWLH1.6, SWLH11.6, SWLH21.6, SWLH31.6, SWLH41.6, SWLH51.6; no longer SWLH1.1, SWLH11.1, SWLH21.1, SWLH31.1, SWLH41.1, SWLH51.1
- net col2: now also SWLH12.6, SWLH2.6, SWLH22.6, SWLH32.6, SWLH42.6, SWLH52.6; no longer SWLH12.1, SWLH2.1, SWLH22.1, SWLH32.1, SWLH42.1, SWLH52.1
- net col3: now also SWLH13.6, SWLH23.6, SWLH3.6, SWLH33.6, SWLH43.6, SWLH53.6; no longer SWLH13.1, SWLH23.1, SWLH3.1, SWLH33.1, SWLH43.1, SWLH53.1
- net col4: now also SWLH14.6, SWLH24.6, SWLH34.6, SWLH4.6, SWLH44.6, SWLH54.6; no longer SWLH14.1, SWLH24.1, SWLH34.1, SWLH4.1, SWLH44.1, SWLH54.1
- net col5: now also SWLH15.6, SWLH25.6, SWLH35.6, SWLH45.6, SWLH5.6, SWLH55.6; no longer SWLH15.1, SWLH25.1, SWLH35.1, SWLH45.1, SWLH5.1, SWLH55.1
- net col6: now also SWLH16.6, SWLH26.6, SWLH36.6, SWLH46.6, SWLH56.6, SWLH6.6; no longer SWLH16.1, SWLH26.1, SWLH36.1, SWLH46.1, SWLH56.1, SWLH6.1
- net col8: now also SWLH18.6, SWLH28.6, SWLH38.6, SWLH48.6, SWLH58.6, SWLH8.6; no longer SWLH18.1, SWLH28.1, SWLH38.1, SWLH48.1, SWLH58.1, SWLH8.1
- net at D2.2 (A): now also SWLH2.5; no longer SWLH2.2
- net at D13.2 (A): now also SWLH13.5; no longer SWLH13.2
- net at D51.2 (A): now also SWLH51.5; no longer SWLH51.2
- net at D43.2 (A): now also SWLH43.5; no longer SWLH43.2
- net at D16.2 (A): now also SWLH16.5; no longer SWLH16.2
- net at D33.2 (A): now also SWLH33.5; no longer SWLH33.2
- net at D50.2 (A): now also SWLH50.5; no longer SWLH50.2
- net at D6.2 (A): now also SWLH6.5; no longer SWLH6.2
- net at D34.2 (A): now also SWLH34.5; no longer SWLH34.2
- net at D48.2 (A): now also SWLH48.5; no longer SWLH48.2
- net at D15.2 (A): now also SWLH15.5; no longer SWLH15.2
- net at D56.2 (A): now also SWLH56.5; no longer SWLH56.2
- net at D22.2 (A): now also SWLH22.5; no longer SWLH22.2
- net at D25.2 (A): now also SWLH25.5; no longer SWLH25.2
- net at D44.2 (A): now also SWLH44.5; no longer SWLH44.2
- net at D38.2 (A): now also SWLH38.5; no longer SWLH38.2
- net at D14.2 (A): now also SWLH14.5; no longer SWLH14.2
- net at D8.2 (A): now also SWLH8.5; no longer SWLH8.2
- net at D18.2 (A): now also SWLH18.5; no longer SWLH18.2
- net at D35.2 (A): now also SWLH35.5; no longer SWLH35.2
- net at D31.2 (A): now also SWLH31.5; no longer SWLH31.2
- net at D26.2 (A): now also SWLH26.5; no longer SWLH26.2
- net at D53.2 (A): now also SWLH53.5; no longer SWLH53.2
- net at D55.2 (A): now also SWLH55.5; no longer SWLH55.2
- net at D11.2 (A): now also SWLH11.5; no longer SWLH11.2
- net at D57.2 (A): now also SWLH57.5; no longer SWLH57.2
- net at D27.2 (A): now also SWLH27.5; no longer SWLH27.2
- net at D7.2 (A): now also SWLH7.5; no longer SWLH7.2
- net at D5.2 (A): now also SWLH5.5; no longer SWLH5.2
- net at D52.2 (A): now also SWLH52.5; no longer SWLH52.2
- net at D3.2 (A): now also SWLH3.5; no longer SWLH3.2
- net at D28.2 (A): now also SWLH28.5; no longer SWLH28.2
- net at D37.2 (A): now also SWLH37.5; no longer SWLH37.2
- net at D21.2 (A): now also SWLH21.5; no longer SWLH21.2
- net at D4.2 (A): now also SWLH4.5; no longer SWLH4.2
- net at D17.2 (A): now also SWLH17.5; no longer SWLH17.2
- net at D36.2 (A): now also SWLH36.5; no longer SWLH36.2
- net at D41.2 (A): now also SWLH41.5; no longer SWLH41.2
- net at D46.2 (A): now also SWLH46.5; no longer SWLH46.2
- net at D1.2 (A): now also SWLH1.5; no longer SWLH1.2
- net at D45.2 (A): now also SWLH45.5; no longer SWLH45.2
- net at D32.2 (A): now also SWLH32.5; no longer SWLH32.2
- net at D42.2 (A): now also SWLH42.5; no longer SWLH42.2
- net at D12.2 (A): now also SWLH12.5; no longer SWLH12.2
- net at D54.2 (A): now also SWLH54.5; no longer SWLH54.2
- net at D58.2 (A): now also SWLH58.5; no longer SWLH58.2
- net at D24.2 (A): now also SWLH24.5; no longer SWLH24.2
- net at D23.2 (A): now also SWLH23.5; no longer SWLH23.2
- new net: SW?.2 (DOUT), SW?.4 (DIN) (x19)
- new net: SW.2 (DOUT), SW?.4 (DIN)
Other:
- moved on the sheet: H1, H10, H11, H2, H3, H4, H5, H6, H7, H8, H9, S1
