File: ergodonk_pcb/ergodonk_pcb.kicad_sch (KiCad schematic)
At the start: 132 parts, among them J1 TRRS, J11 Pimaroni Trackball, Q1 TIP120, SW08_RH10 SW_PUSH_LED, SW1 SW_PUSH_LED, SW10 SW_PUSH_LED, SW11 SW_PUSH_LED, SW12 SW_PUSH_LED, SW13 SW_PUSH_LED, SW14 SW_PUSH_LED, SW15 SW_PUSH_LED, SW16 SW_PUSH_LED, SW17 SW_PUSH_LED, SW18_RH10 SW_PUSH_LED, SW2 SW_PUSH_LED, SW20 SW_PUSH_LED, SW21 SW_PUSH_LED, SW22 SW_PUSH_LED, SW23 SW_PUSH_LED, SW24 SW_PUSH_LED, SW25 SW_PUSH_LED, SW26 SW_PUSH_LED, SW27 SW_PUSH_LED, SW28_RH10 SW_PUSH_LED, SW3 SW_PUSH_LED, SW30 SW_PUSH_LED, SW31 SW_PUSH_LED, SW32 SW_PUSH_LED, SW33 SW_PUSH_LED, SW34 SW_PUSH_LED, SW35 SW_PUSH_LED, SW36 SW_PUSH_LED, SW37 SW_PUSH_LED, SW38_RH10 SW_PUSH_LED, SW4 SW_PUSH_LED, SW40 SW_PUSH_LED, SW42 SW_PUSH_LED, SW43 SW_PUSH_LED, SW44 SW_PUSH_LED, SW45 SW_PUSH_LED, SW46 SW_PUSH_LED, SW47 SW_PUSH_LED, SW48_RH10 SW_PUSH_LED, SW5 SW_PUSH_LED, SW50 SW_PUSH_LED, SW51 SW_PUSH_LED, SW52 SW_PUSH_LED, SW53 SW_PUSH_LED, SW54 SW_PUSH_LED, SW55 SW_PUSH_LED, SW56 SW_PUSH_LED, SW57 SW_PUSH_LED, SW58 SW_PUSH_LED, SW6 SW_PUSH_LED, SW7 SW_PUSH_LED, U10 Pico

Commit message: Rewired to VBus for 5V and updated dsn
Parts:
- removed R1: 5k6, Resistor_SMD:R_1206_3216Metric_Pad1.30x1.75mm_HandSolder, symbol Device:R
- removed R2: 10k, Resistor_SMD:R_1206_3216Metric_Pad1.30x1.75mm_HandSolder, symbol Device:R
Connections:
- net VCC: now also U10.40 (VBUS); no longer U10.37 (3V3_EN)
Other:
- note removed: "??? Power???"
Changed lines of the file:
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@@
   (junction (at 313.69 100.33) (diameter 0) (color 0 0 0 0)
   )
-  (junction (at 68.58 179.07) (diameter 0) (color 0 0 0 0)
-  )
   (junction (at 313.69 78.74) (diameter 0) (color 0 0 0 0)
   )
@@
   (junction (at 210.82 223.52) (diameter 0) (color 0 0 0 0)
   )
+  (junction (at 68.58 176.53) (diameter 0) (color 0 0 0 0)
+  )
   (junction (at 285.75 129.54) (diameter 0) (color 0 0 0 0)
   )
@@
   (junction (at 285.75 86.36) (diameter 0) (color 0 0 0 0)
   )
-  (junction (at 452.12 95.25) (diameter 0) (color 0 0 0 0)
-  )
   (junction (at 307.34 86.36) (diameter 0) (color 0 0 0 0)
   )
@@
     (stroke (width 0) (type default))
   )
-  (wire (pts (xy 68.58 179.07) (xy 68.58 187.96))
+  (wire (pts (xy 68.58 176.53) (xy 68.58 180.34))
     (stroke (width 0) (type default))
   )
@@
     (stroke (width 0) (type default))
   )
+  (wire (pts (xy 62.23 180.34) (xy 68.58 180.34))
+    (stroke (width 0) (type default))
+  )
   (wire (pts (xy 39.37 55.88) (xy 39.37 72.39))
     (stroke (width 0) (type default))
@@
     (stroke (width 0) (type default))
   )
+  (wire (pts (xy 68.58 176.53) (xy 74.93 176.53))
+    (stroke (width 0) (type default))
+  )
   (wire (pts (xy 55.88 72.39) (xy 62.23 72.39))
     (stroke (width 0) (type default))
@@
     (stroke (width 0) (type default))
   )
-  (wire (pts (xy 68.58 179.07) (xy 74.93 179.07))
-    (stroke (width 0) (type default))
-  )
   (polyline (pts (xy 210.82 152.4) (xy 121.92 152.4))
     (stroke (width 0) (type default))
@@
     (stroke (width 0) (type default))
   )
-  (wire (pts (xy 452.12 95.25) (xy 461.01 95.25))
-    (stroke (width 0) (type default))
-  )
   (polyline (pts (xy 163.83 240.03) (xy 193.04 240.03))
     (stroke (width 0) (type default))
@@
     (stroke (width 0) (type default))
   )
-  (wire (pts (xy 62.23 187.96) (xy 68.58 187.96))
-    (stroke (width 0) (type default))
-  )
   (wire (pts (xy 165.1 93.98) (xy 158.75 93.98))
     (stroke (width 0) (type default))
@@
     (fill (type none))
   )
-  (rectangle (start 54.61 167.64) (end 96.52 191.77)
-    (stroke (width 0) (type default))
-    (fill (type none))
-  )
   (rectangle (start 198.12 168.91) (end 250.19 193.04)
     (stroke (width 0) (type default))
@@
     (effects (font (size 1.27 1.27)) (justify left bottom))
   )
-  (text "??? Power???" (at 55.88 173.99 0)
-    (effects (font (size 1.27 1.27)) (justify left bottom))
-  )
   (text "Rotary Encoder" (at 165.1 107.95 0)
     (effects (font (size 1.27 1.27)) (justify left bottom))
@@
     )
   )
-  (global_label "vbus_sense" (shape input) (at 461.01 95.25 0) (fields_autoplaced)
-    (effects (font (size 1.27 1.27)) (justify left))
-    (property "Intersheetrefs" "${INTERSHEET_REFS}" (at 474.0669 95.1706 0)
-      (effects (font (size 1.27 1.27)) (justify left) hide)
-    )
-  )
   (global_label "row0" (shape input) (at 219.71 43.18 180) (fields_autoplaced)
     (effects (font (size 1.27 1.27)) (justify right))
@@
     )
   )
-  (symbol (lib_id "power:VCC") (at 68.58 179.07 0) (unit 1)
-    (in_bom yes) (on_board yes) (dnp no) (fields_autoplaced)
-    (property "Reference" "#PWR021" (at 68.58 182.88 0)
+  (symbol (lib_id "power:VCC") (at 68.58 176.53 0) (unit 1)
+    (in_bom yes) (on_board yes) (dnp no)
+    (property "Reference" "#PWR021" (at 68.58 180.34 0)
       (effects (font (size 1.27 1.27)) hide)
     )
-    (property "Value" "VCC" (at 68.58 175.26 0)
+    (property "Value" "VCC" (at 68.58 172.72 0)
       (effects (font (size 1.27 1.27)))
     )
-    (property "Footprint" "" (at 68.58 179.07 0)
+    (property "Footprint" "" (at 68.58 176.53 0)
       (effects (font (size 1.27 1.27)) hide)
     )
-    (property "Datasheet" "" (at 68.58 179.07 0)
+    (property "Datasheet" "" (at 68.58 176.53 0)
       (effects (font (size 1.27 1.27)) hide)
     )
@@
     )
   )
-  (symbol (lib_id "Device:R") (at 452.12 99.06 0) (unit 1)
-    (in_bom yes) (on_board yes) (dnp no) (fields_autoplaced)
-    (property "Reference" "R2" (at 454.66 97.7899 0)
-      (effects (font (size 1.27 1.27)) (justify left))
-    )
-    (property "Value" "10k" (at 454.66 100.3299 0)
-      (effects (font (size 1.27 1.27)) (justify left))
-    )
-    (property "Footprint" "Resistor_SMD:R_1206_3216Metric_Pad1.30x1.75mm_HandSolder" (at 450.342 99.06 90)
-      (effects (font (size 1.27 1.27)) hide)
-    )
-    (property "Datasheet" "~" (at 452.12 99.06 0)
-      (effects (font (size 1.27 1.27)) hide)
-    )
-    (pin "1")
-    (pin "2")
-    (instances
-      (project "keyboard_pcb"
-        (path "/9538e4ed-27e6-4c37-b989-9859dc0d49e8"
-          (reference "R2") (unit 1)
-        )
-      )
-      (project "ergodonk_pcb"
-        (path "/ed1aaf15-4e1f-4159-b371-d99b3fb972ad"
-          (reference "R11") (unit 1)
-        )
-      )
-    )
-  )
   (symbol (lib_id "Device:D") (at 307.34 147.32 90) (unit 1)
     (in_bom yes) (on_board yes) (dnp no) (fields_autoplaced)
@@
     )
   )
-  (symbol (lib_id "Device:R") (at 452.12 91.44 0) (unit 1)
-    (in_bom yes) (on_board yes) (dnp no) (fields_autoplaced)
-    (property "Reference" "R1" (at 454.66 90.1699 0)
-      (effects (font (size 1.27 1.27)) (justify left))
-    )
-    (property "Value" "5k6" (at 454.66 92.7099 0)
-      (effects (font (size 1.27 1.27)) (justify left))
-    )
-    (property "Footprint" "Resistor_SMD:R_1206_3216Metric_Pad1.30x1.75mm_HandSolder" (at 450.342 91.44 90)
-      (effects (font (size 1.27 1.27)) hide)
-    )
-    (property "Datasheet" "~" (at 452.12 91.44 0)
-      (effects (font (size 1.27 1.27)) hide)
-    )
-    (pin "1")
-    (pin "2")
-    (instances
-      (project "keyboard_pcb"
-        (path "/9538e4ed-27e6-4c37-b989-9859dc0d49e8"
-          (reference "R1") (unit 1)
-        )
-      )
-      (project "ergodonk_pcb"
-        (path "/ed1aaf15-4e1f-4159-b371-d99b3fb972ad"
-          (reference "R10") (unit 1)
-        )
-      )
-    )
-  )
   (symbol (lib_id "Mechanical:MountingHole") (at -250.19 416.56 0) (unit 1)
     (in_bom yes) (on_board yes) (dnp no) (fields_autoplaced)
@@
     )
   )
-  (symbol (lib_id "power:GND") (at 452.12 102.87 0) (unit 1)
-    (in_bom yes) (on_board yes) (dnp no) (fields_autoplaced)
-    (property "Reference" "#PWR0127" (at 452.12 109.22 0)
-      (effects (font (size 1.27 1.27)) hide)
-    )
-    (property "Value" "GND" (at 454.66 104.1399 0)
-      (effects (font (size 1.27 1.27)) (justify left))
-    )
-    (property "Footprint" "" (at 452.12 102.87 0)
-      (effects (font (size 1.27 1.27)) hide)
-    )
-    (property "Datasheet" "" (at 452.12 102.87 0)
-      (effects (font (size 1.27 1.27)) hide)
-    )
-    (pin "1")
-    (instances
-      (project "keyboard_pcb"
-        (path "/9538e4ed-27e6-4c37-b989-9859dc0d49e8"
-          (reference "#PWR0127") (unit 1)
-        )
-      )
-      (project "ergodonk_pcb"
-        (path "/ed1aaf15-4e1f-4159-b371-d99b3fb972ad"
-          (reference "#PWR014") (unit 1)
-        )
-      )
-    )
-  )
   (symbol (lib_id "SofleKeyboard:SW_PUSH_LED") (at 132.08 74.93 0) (mirror y) (unit 2)
     (in_bom yes) (on_board yes) (dnp no)
@@
     )
   )
-  (symbol (lib_id "power:VBUS") (at 452.12 87.63 0) (unit 1)
-    (in_bom yes) (on_board yes) (dnp no) (fields_autoplaced)
-    (property "Reference" "#PWR0125" (at 452.12 91.44 0)
-      (effects (font (size 1.27 1.27)) hide)
-    )
-    (property "Value" "VBUS" (at 452.12 82.55 0)
-      (effects (font (size 1.27 1.27)))
-    )
-    (property "Footprint" "" (at 452.12 87.63 0)
-      (effects (font (size 1.27 1.27)) hide)
-    )
-    (property "Datasheet" "" (at 452.12 87.63 0)
-      (effects (font (size 1.27 1.27)) hide)
-    )
-    (pin "1")
-    (instances
-      (project "keyboard_pcb"
-        (path "/9538e4ed-27e6-4c37-b989-9859dc0d49e8"
-          (reference "#PWR0125") (unit 1)
-        )
-      )
-      (project "ergodonk_pcb"
-        (path "/ed1aaf15-4e1f-4159-b371-d99b3fb972ad"
-          (reference "#PWR013") (unit 1)
-        )
-      )
-    )
-  )
   (symbol (lib_id "Device:D") (at 307.34 60.96 90) (unit 1)
     (in_bom yes) (on_board yes) (dnp no) (fields_autoplaced)
@@
     )
   )
-  (symbol (lib_id "power:PWR_FLAG") (at 74.93 179.07 0) (unit 1)
+  (symbol (lib_id "power:PWR_FLAG") (at 74.93 176.53 0) (unit 1)
     (in_bom yes) (on_board yes) (dnp no)
-    (property "Reference" "#FLG011" (at 74.93 177.165 0)
+    (property "Reference" "#FLG011" (at 74.93 174.625 0)
       (effects (font (size 1.27 1.27)) hide)
     )
-    (property "Value" "PWR_FLAG" (at 74.93 173.99 0)
+    (property "Value" "PWR_FLAG" (at 74.93 171.45 0)
       (effects (font (size 1.27 1.27)))
     )
-    (property "Footprint" "" (at 74.93 179.07 0)
+    (property "Footprint" "" (at 74.93 176.53 0)
       (effects (font (size 1.27 1.27)) hide)
     )
-    (property "Datasheet" "~" (at 74.93 179.07 0)
+    (property "Datasheet" "~" (at 74.93 176.53 0)
       (effects (font (size 1.27 1.27)) hide)
     )

Commit message: Mounting hole realingmngment for top plate
Parts:
- added H12, H13: MountingHole, MountingHole:MountingHole_2.2mm_M2_Pad_Via, symbol Mechanical:MountingHole
Other:
- moved on the sheet: H1, H10, H11, H2, H3, H4, H5, H6, H7, H8, H9, S1
