File: ergodonk_pico/ergodonk_pico.kicad_sch (KiCad schematic)
At the start: 131 parts, among them J2 Pimaroni Trackball, J3 AudioJack4, Q1 TIP120, SW08_RH1 SW_PUSH_LED, SW1 SW_PUSH_LED, SW10 SW_PUSH_LED, SW11 SW_PUSH_LED, SW12 SW_PUSH_LED, SW13 SW_PUSH_LED, SW14 SW_PUSH_LED, SW15 SW_PUSH_LED, SW16 SW_PUSH_LED, SW17 SW_PUSH_LED, SW18 SW_PUSH_LED, SW18_RH1 SW_PUSH_LED, SW19 SW_PUSH_LED, SW2 SW_PUSH_LED, SW20 SW_PUSH_LED, SW21 SW_PUSH_LED, SW22 SW_PUSH_LED, SW23 SW_PUSH_LED, SW24 SW_PUSH_LED, SW25 SW_PUSH_LED, SW26 SW_PUSH_LED, SW27 SW_PUSH_LED, SW28 SW_PUSH_LED, SW28_RH1 SW_PUSH_LED, SW29 SW_PUSH_LED, SW3 SW_PUSH_LED, SW30 SW_PUSH_LED, SW31 SW_PUSH_LED, SW32 SW_PUSH_LED, SW33 SW_PUSH_LED, SW34 SW_PUSH_LED, SW35 SW_PUSH_LED, SW36 SW_PUSH_LED, SW37 SW_PUSH_LED, SW38 SW_PUSH_LED, SW38_RH1 SW_PUSH_LED, SW39 SW_PUSH_LED, SW4 SW_PUSH_LED, SW40 SW_PUSH_LED, SW41 SW_PUSH_LED, SW42 SW_PUSH_LED, SW43 SW_PUSH_LED, SW44 SW_PUSH_LED, SW45 SW_PUSH_LED, SW46 SW_PUSH_LED, SW47 SW_PUSH_LED, SW48_RH1 SW_PUSH_LED, SW5 SW_PUSH_LED, SW6 SW_PUSH_LED, SW7 SW_PUSH_LED, SW8 SW_PUSH_LED, SW9 SW_PUSH_LED, U2 Pico

Commit message: Ergodonk pico schematic  update
Parts:
- removed D08_RH1, D18_RH1, D28_RH1, D38_RH1: D, ergodonk_pico:D3_TH_SMD_v2, symbol Device:D
- removed unit 1 of SW08_RH1
- removed unit 1 of SW18_RH1
- removed unit 1 of SW28_RH1
- removed unit 1 of SW38_RH1
- removed unit 1 of SW48_RH1
- added D49, D50, D51, D52, D53, D54, D55, D56, D57, D58, D59, D60, D61, D62, D63, D64, D65 (x2), D66, D67, D68, D69, D70, D71, D72, D73, D74, D75, D76, D77, D78, D79, D80, D81 (x2), D82 (x2), D83, D84, D85, D86, D87, D88, D89, D90, D91, D92, D93, D94, D95, D96, D97: D, ergodonk_pico:D3_TH_SMD_v2, symbol Device:D
- added SW48_RH2, SW49, SW50, SW51, SW52, SW53, SW54, SW55, SW56, SW57, SW58, SW59, SW60, SW61, SW62, SW63, SW64, SW65 (x2), SW66, SW67, SW68, SW69, SW70, SW71, SW72, SW73, SW74, SW75, SW76, SW77, SW78, SW79, SW80 (x2), SW81 (x2), SW82 (x2), SW83 (x2), SW84, SW85, SW86, SW87, SW88, SW89, SW90, SW91, SW92, SW93, SW94: SW_Push, symbol Switch:SW_Push
- added SWRH_ROT1: RotaryEncoder_Switch, ergodonk_kicad_library:RotaryEncoder_EC11_ergodonk_variant, symbol Device:RotaryEncoder_Switch
- SW1, SW10, SW11, SW12, SW13, SW14, SW15, SW16, SW17, SW18, SW19, SW2, SW20, SW21, SW22, SW23, SW24, SW25, SW26, SW27, SW28, SW29, SW3, SW30, SW31, SW32, SW33, SW34, SW35, SW36, SW37, SW4, SW5, SW6, SW7, SW8, SW9: value SW_PUSH_LED -> SW_Push; footprint ergodonk_kicad_library:Chunky_2040_footprint_ergodonk_customs -> (none); symbol Ergodonk_symbols:SW_PUSH_LED -> Switch:SW_Push; LCSC (none) -> C5156480
- SW39: renamed from SW38; value SW_PUSH_LED -> SW_Push; footprint ergodonk_kicad_library:Chunky_2040_footprint_ergodonk_customs -> (none); symbol Ergodonk_symbols:SW_PUSH_LED -> Switch:SW_Push; LCSC (none) -> C5156480
- SW40: renamed from SW39; value SW_PUSH_LED -> SW_Push; footprint ergodonk_kicad_library:Chunky_2040_footprint_ergodonk_customs -> (none); symbol Ergodonk_symbols:SW_PUSH_LED -> Switch:SW_Push; LCSC (none) -> C5156480
- SW41: renamed from SW40; value SW_PUSH_LED -> SW_Push; footprint ergodonk_kicad_library:Chunky_2040_footprint_ergodonk_customs -> (none); symbol Ergodonk_symbols:SW_PUSH_LED -> Switch:SW_Push; LCSC (none) -> C5156480
- SW42: renamed from SW41; value SW_PUSH_LED -> SW_Push; footprint ergodonk_kicad_library:Chunky_2040_footprint_ergodonk_customs -> (none); symbol Ergodonk_symbols:SW_PUSH_LED -> Switch:SW_Push; LCSC (none) -> C5156480
- SW43: renamed from SW42; value SW_PUSH_LED -> SW_Push; footprint ergodonk_kicad_library:Chunky_2040_footprint_ergodonk_customs -> (none); symbol Ergodonk_symbols:SW_PUSH_LED -> Switch:SW_Push; LCSC (none) -> C5156480
- SW44: renamed from SW43; value SW_PUSH_LED -> SW_Push; footprint ergodonk_kicad_library:Chunky_2040_footprint_ergodonk_customs -> (none); symbol Ergodonk_symbols:SW_PUSH_LED -> Switch:SW_Push; LCSC (none) -> C5156480
- SW45: renamed from SW44; value SW_PUSH_LED -> SW_Push; footprint ergodonk_kicad_library:Chunky_2040_footprint_ergodonk_customs -> (none); symbol Ergodonk_symbols:SW_PUSH_LED -> Switch:SW_Push; LCSC (none) -> C5156480
- SW46: renamed from SW45; value SW_PUSH_LED -> SW_Push; footprint ergodonk_kicad_library:Chunky_2040_footprint_ergodonk_customs -> (none); symbol Ergodonk_symbols:SW_PUSH_LED -> Switch:SW_Push; LCSC (none) -> C5156480
- SW47: renamed from SW46; value SW_PUSH_LED -> SW_Push; footprint ergodonk_kicad_library:Chunky_2040_footprint_ergodonk_customs -> (none); symbol Ergodonk_symbols:SW_PUSH_LED -> Switch:SW_Push; LCSC (none) -> C5156480
- SW48: renamed from SW47; value SW_PUSH_LED -> SW_Push; footprint ergodonk_kicad_library:Chunky_2040_footprint_ergodonk_customs -> (none); symbol Ergodonk_symbols:SW_PUSH_LED -> Switch:SW_Push; LCSC (none) -> C5156480
Connections:
- net GND: now also SWRH_ROT1.C
- net col0: no longer SW15.6, SW23.6, SW31.6, SW39.6, SW48.6
- net col2: no longer SW13.6, SW21.6, SW29.6, SW37.6, SW46.6, SW6.6
- net col3: no longer SW12.6, SW20.6, SW28.6, SW36.6, SW45.6, SW5.6
- net col4: no longer SW11.6, SW19.6, SW27.6, SW35.6, SW4.6, SW44.6
- net col5: no longer SW10.6, SW18.6, SW26.6, SW3.6, SW34.6, SW43.6
- net col6: no longer SW17.6, SW2.6, SW25.6, SW33.6, SW42.6, SW9.6
- net col7: no longer SW1.6, SW16.6, SW24.6, SW32.6, SW41.6, SW8.6
- net col8: no longer SW40.6
- net encA: now also SWRH_ROT1.A
- net encB: now also SWRH_ROT1.B
- net row0: now also D49.1 (K), D50.1 (K), D51.1 (K), D52.1 (K), D53.1 (K), D54.1 (K), D55.1 (K), D56.1 (K)
- net row1: now also D57.1 (K), D58.1 (K), D59.1 (K), D60.1 (K), D61.1 (K), D62.1 (K), D63.1 (K), D64.1 (K), D65.1 (K)
- net row2: now also D65.1 (K), D66.1 (K), D67.1 (K), D68.1 (K), D69.1 (K), D70.1 (K), D71.1 (K), D72.1 (K), D73.1 (K)
- net row3: now also D74.1 (K), D75.1 (K), D76.1 (K), D77.1 (K), D78.1 (K), D79.1 (K), D80.1 (K), D81.1 (K), D82.1 (K)
- net row4: now also D81.1 (K), D82.1 (K), D83.1 (K), D84.1 (K), D85.1 (K), D86.1 (K), D87.1 (K), D88.1 (K)
- net row5: now also D89.1 (K), D90.1 (K), D91.1 (K), D92.1 (K), D93.1 (K), D94.1 (K), D95.1 (K), D96.1 (K), D97.1 (K)
- net at D3.2 (A): no longer SW3.5
- net at D21.2 (A): no longer SW21.5
- net at D13.2 (A): no longer SW13.5
- net at D41.2 (A): no longer SW41.5
- net at D7.2 (A): no longer SW7.5
- net at D44.2 (A): no longer SW44.5
- net at D36.2 (A): no longer SW36.5
- net at D14.2 (A): no longer SW14.5
- net at D47.2 (A): no longer SW47.5
- net at D23.2 (A): no longer SW23.5
- net at D40.2 (A): no longer SW40.5
- net at D33.2 (A): no longer SW33.5
- net at D11.2 (A): no longer SW11.5
- net at D30.2 (A): no longer SW30.5
- net at D35.2 (A): no longer SW35.5
- net at D4.2 (A): no longer SW4.5
- net at D31.2 (A): no longer SW31.5
- net at D1.2 (A): no longer SW1.5
- net at D28.2 (A): no longer SW28.5
- net at D39.2 (A): no longer SW39.5
- net at D22.2 (A): no longer SW22.5
- net at D9.2 (A): no longer SW9.5
- net at D16.2 (A): no longer SW16.5
- net at D27.2 (A): no longer SW27.5
- net at D8.2 (A): no longer SW8.5
- net at D45.2 (A): no longer SW45.5
- net at D29.2 (A): no longer SW29.5
- net at D34.2 (A): no longer SW34.5
- net at D32.2 (A): no longer SW32.5
- net at D42.2 (A): no longer SW42.5
- net at D37.2 (A): no longer SW37.5
- net at D10.2 (A): no longer SW10.5
- net at D12.2 (A): no longer SW12.5
- net at D6.2 (A): no longer SW6.5
- net at D24.2 (A): no longer SW24.5
- net at D46.2 (A): no longer SW46.5
- net at D5.2 (A): no longer SW5.5
- net at D26.2 (A): no longer SW26.5
- net at D43.2 (A): no longer SW43.5
- net at D18.2 (A): no longer SW18.5
- net at D17.2 (A): no longer SW17.5
- net at D2.2 (A): no longer SW2.5
- net at D15.2 (A): no longer SW15.5
- net at D48.2 (A): no longer SW48.5
- net at D25.2 (A): no longer SW25.5
- net at D20.2 (A): no longer SW20.5
- net at D19.2 (A): no longer SW19.5
- removed net SW41A: SW14.6, SW22.6, SW30.6, SW47.6, SW7.6, SWLH_ROT1.S1, U2.12 (GPIO9)
- net SW41B renamed SW38B
- new net SW38A: SWLH_ROT1.S1, SWRH_ROT1.S1, U2.12 (GPIO9)
- new net SW_RH_ROT_B: D82.2 (A), SWRH_ROT1.S2
Other:
- note added: "Rotary Knob LH"
- note added: "Rotary Knob RH"
- note removed: "Rotary Knob"
- moved on the sheet: D1, D10, D11, D12, D13, D14, D15, D16, D17, D18, D19, D2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

Commit message: Updated pico RH schematics
Parts:
- renumbered D96 to D100, D97 to D101, D65 to D66, D66 to D67, D67 to D68, D68 to D69, D69 to D70, D70 to D71, D71 to D72, D72 to D73, D73 to D74, D74 to D75, D75 to D76, D76 to D77, D77 to D78, D78 to D79, D79 to D80, D80 to D81, D81 to D82, D82 to D83, D81 to D84, D82 to D85, D83 to D86, D84 to D87, D85 to D88, D86 to D89, D87 to D90, D88 to D91, D48_RH1 to D92, D89 to D93, D90 to D94, D91 to D95, D92 to D96, D93 to D97, D94 to D98, D95 to D99, SW93 to SW100, SW94 to SW101, SW65 to SW66, SW66 to SW67, SW67 to SW68, SW68 to SW69, SW69 to SW70, SW70 to SW71, SW71 to SW72, SW72 to SW73, SW73 to SW74, SW74 to SW75, SW75 to SW76, SW76 to SW77, SW77 to SW78, SW78 to SW79, SW79 to SW80, SW80 to SW81, SW81 to SW82, SW82 to SW83, SW83 to SW84, SW80 to SW86, SW81 to SW87, SW82 to SW88, SW83 to SW89, SW84 to SW90, SW85 to SW91, SW48_RH2 to SW92, SW86 to SW93, SW87 to SW94, SW88 to SW95, SW89 to SW96, SW90 to SW97, SW91 to SW98, SW92 to SW99
Connections:
- net SW38A is gone; now on net SW38_A: SWLH_ROT1.S1, SWRH_ROT1.S1, U2.12 (GPIO9)
- net col0: now also SW15.1, SW23.1, SW31.1, SW39.1, SW48.1, SW57.1, SW66.1, SW75.1, SW84.1, SW93.1
- net col2: now also SW13.1, SW21.1, SW29.1, SW37.1, SW46.1, SW50.1, SW59.1, SW6.1, SW68.1, SW77.1, SW86.1, SW95.1
- net col3: now also SW12.1, SW20.1, SW28.1, SW36.1, SW45.1, SW5.1, SW51.1, SW60.1, SW69.1, SW78.1, SW87.1, SW96.1
- net col4: now also SW11.1, SW19.1, SW27.1, SW35.1, SW4.1, SW44.1, SW52.1, SW61.1, SW70.1, SW79.1, SW88.1, SW97.1
- net col5: now also SW10.1, SW18.1, SW26.1, SW3.1, SW34.1, SW43.1, SW53.1, SW62.1, SW71.1, SW80.1, SW89.1, SW98.1
- net col6: now also SW17.1, SW2.1, SW25.1, SW33.1, SW42.1, SW54.1, SW63.1, SW72.1, SW81.1, SW9.1, SW90.1, SW99.1
- net col7: now also SW1.1, SW100.1, SW16.1, SW24.1, SW32.1, SW41.1, SW55.1, SW64.1, SW73.1, SW8.1, SW82.1, SW91.1
- net col8: now also SW101.1, SW40.1, SW56.1, SW65.1, SW74.1, SW83.1, SW92.1
- net at D3.2 (A): now also SW3.2
- net at D93.2 (A): now also SW93.2
- net at D63.2 (A): now also SW63.2
- net at SW52.2: now also D52.2 (A)
- net at D21.2 (A): now also SW21.2
- net at D78.2 (A): now also SW78.2
- net at SW59.2: now also D59.2 (A)
- net at D94.2 (A): now also SW94.2
- net at SW62.2: now also D62.2 (A)
- net at SW77.2: now also D77.2 (A)
- net at SW90.2: now also D90.2 (A)
- net at D13.2 (A): now also SW13.2
- net at D41.2 (A): now also SW41.2
- net at D99.2 (A): now also SW99.2
- net SW38_A: now reaches SW7.1
- net SW38_A: now also SW14.1, SW22.1, SW30.1, SW47.1, SW49.1, SW58.1, SW67.1, SW76.1, SW94.1
- net at SW7.2: now also D7.2 (A)
- net at SW100.2: now also D100.2 (A)
- net at D61.2 (A): now also SW61.2
- net at SW44.2: now also D44.2 (A)
- net at D36.2 (A): now also SW36.2
- net at SW14.2: now also D14.2 (A)
- net at SW58.2: now also D58.2 (A)
- net at D47.2 (A): now also SW47.2
- net at D70.2 (A): now also SW70.2
- net at D23.2 (A): now also SW23.2
- net at SW82.2: now also D82.2 (A)
- net at SW83.2: now also D83.2 (A)
- net at D40.2 (A): now also SW40.2
- net at D84.2 (A): now also SW84.2
- net at SW50.2: now also D50.2 (A)
- net at D79.2 (A): now also SW79.2
- net at SW33.2: now also D33.2 (A)
- net at D71.2 (A): now also SW71.2
- net at SW11.2: now also D11.2 (A)
- net at D81.2 (A): now also SW81.2
- net at SW80.2: now also D80.2 (A)
- net at SW56.2: now also D56.2 (A)
- net at SW30.2: now also D30.2 (A)
- net at SW72.2: now also D72.2 (A)
- net at D68.2 (A): now also SW68.2
- net at D97.2 (A): now also SW97.2
- net at D35.2 (A): now also SW35.2
- net at SW4.2: now also D4.2 (A)
- net at D31.2 (A): now also SW31.2
- net at SW1.2: now also D1.2 (A)
- net at SW54.2: now also D54.2 (A)
- net at SW66.2: now also D66.2 (A)
- net at D28.2 (A): now also SW28.2
- net at D69.2 (A): now also SW69.2
- net at SW39.2: now also D39.2 (A)
- net at SW22.2: now also D22.2 (A)
- net at D96.2 (A): now also SW96.2
- net at SW9.2: now also D9.2 (A)
- net at D16.2 (A): now also SW16.2
- net at SW27.2: now also D27.2 (A)
- net at SW8.2: now also D8.2 (A)
- net at D45.2 (A): now also SW45.2
- net at D29.2 (A): now also SW29.2
- net at SW60.2: now also D60.2 (A)
- net at SW65.2: now also D65.2 (A)
- net at SW64.2: now also D64.2 (A)
- net at SW76.2: now also D76.2 (A)
- net at D34.2 (A): now also SW34.2
- net at SW101.2: now also D101.2 (A)
- net at D74.2 (A): now also SW74.2
- net at SW98.2: now also D98.2 (A)
- net at D32.2 (A): now also SW32.2
- net at D42.2 (A): now also SW42.2
- net at D57.2 (A): now also SW57.2
- net at D55.2 (A): now also SW55.2
- net at SW37.2: now also D37.2 (A)
- net at SW53.2: now also D53.2 (A)
- net at SW49.2: now also D49.2 (A)
- net at D10.2 (A): now also SW10.2
- net at D67.2 (A): now also SW67.2
- net at SW12.2: now also D12.2 (A)
- net at D6.2 (A): now also SW6.2
- net at D24.2 (A): now also SW24.2
- net at D86.2 (A): now also SW86.2
- net at D46.2 (A): now also SW46.2
- net at D5.2 (A): now also SW5.2
- net at SW26.2: now also D26.2 (A)
- net at SW95.2: now also D95.2 (A)
- net at D88.2 (A): now also SW88.2
- net at D43.2 (A): now also SW43.2
- net at D18.2 (A): now also SW18.2
- net at SW17.2: now also D17.2 (A)
- net at SW2.2: now also D2.2 (A)
- net at SW15.2: now also D15.2 (A)
- net at D48.2 (A): now also SW48.2
- net at SW25.2: now also D25.2 (A)
- net at D89.2 (A): now also SW89.2
- net at D20.2 (A): now also SW20.2
- net at D75.2 (A): now also SW75.2
- net at D73.2 (A): now also SW73.2
- net at D19.2 (A): now also SW19.2
- net at SW87.2: now also D87.2 (A)
- net at D91.2 (A): now also SW91.2
- net at D51.2 (A): now also SW51.2
- net SW38B renamed SW38_B
- net SW_RH_ROT_B renamed SW85_B

Commit message: Checkpoint commit
Parts:
- added L1, L10, L11, L12, L13, L14, L15, L16, L17, L18, L19, L2, L20, L21, L22, L23, L24, L25, L26, L27, L28, L29, L3, L30, L31, L32, L33, L34, L35, L36, L37, L38, L39, L4, L40, L41, L42, L43, L44, L45, L46, L47, L48, L5, L6, L7, L8, L9: SK6812MINI-E, ergodonk_pico:SK6812-MINI-E, symbol Ergodonk_symbols:SK6812MINI
- renumbered D49 to D102
Connections:
- net VCC is gone; now on net GND: D102.1 (K), D_SOL_1.C, J2.1 (Pin_1), J3.T, J_SOL_1.2 (Pin_2), OL1.3 (VCC), SW08_RH1.1 (VDD), SW1.1 (VDD), SW10.1 (VDD), SW11.1 (VDD), SW12.1 (VDD), SW13.1 (VDD), SW14.1 (VDD), SW15.1 (VDD), SW16.1 (VDD), SW17.1 (VDD), SW18.1 (VDD), SW18_RH1.1 (VDD), SW19.1 (VDD), SW2.1 (VDD), SW20.1 (VDD), SW21.1 (VDD), SW22.1 (VDD), SW23.1 (VDD), SW24.1 (VDD), SW25.1 (VDD), SW26.1 (VDD), SW27.1 (VDD), SW28.1 (VDD), SW28_RH1.1 (VDD), SW29.1 (VDD), SW3.1 (VDD), SW30.1 (VDD), SW31.1 (VDD), SW32.1 (VDD), SW33.1 (VDD), SW34.1 (VDD), SW35.1 (VDD), SW36.1 (VDD), SW37.1 (VDD), SW38.1 (VDD), SW38_RH1.1 (VDD), SW39.1 (VDD), SW4.1 (VDD), SW40.1 (VDD), SW41.1 (VDD), SW42.1 (VDD), SW43.1 (VDD), SW44.1 (VDD), SW45.1 (VDD), SW46.1 (VDD), SW47.1 (VDD), SW48_RH1.1 (VDD), SW5.1 (VDD), SW6.1 (VDD), SW7.1 (VDD), SW8.1 (VDD), SW9.1 (VDD), U2.39 (VSYS)
- net GND: now also L1.1 (VDD), L1.3 (GND), L10.1 (VDD), L10.3 (GND), L11.1 (VDD), L11.3 (GND), L12.1 (VDD), L12.3 (GND), L13.1 (VDD), L13.3 (GND), L14.1 (VDD), L14.3 (GND), L15.1 (VDD), L15.3 (GND), L16.1 (VDD), L16.3 (GND), L17.1 (VDD), L17.3 (GND), L18.1 (VDD), L18.3 (GND), L19.1 (VDD), L19.3 (GND), L2.1 (VDD), L2.3 (GND), L20.1 (VDD), L20.3 (GND), L21.1 (VDD), L21.3 (GND), L22.1 (VDD), L22.3 (GND), L23.1 (VDD), L23.3 (GND), L24.1 (VDD), L24.3 (GND), L25.1 (VDD), L25.3 (GND), L26.1 (VDD), L26.3 (GND), L27.1 (VDD), L27.3 (GND), L28.1 (VDD), L28.3 (GND), L29.1 (VDD), L29.3 (GND), L3.1 (VDD), L3.3 (GND), L30.1 (VDD), L30.3 (GND), L31.1 (VDD), L31.3 (GND), L32.1 (VDD), L32.3 (GND), L33.1 (VDD), L33.3 (GND), L34.1 (VDD), L34.3 (GND), L35.1 (VDD), L35.3 (GND), L36.1 (VDD), L36.3 (GND), L37.1 (VDD), L37.3 (GND), L38.1 (VDD), L38.3 (GND), L39.1 (VDD), L39.3 (GND), L4.1 (VDD), L4.3 (GND), L40.1 (VDD), L40.3 (GND), L41.1 (VDD), L41.3 (GND), L42.1 (VDD), L42.3 (GND), L43.1 (VDD), L43.3 (GND), L44.1 (VDD), L44.3 (GND), L45.1 (VDD), L45.3 (GND), L46.1 (VDD), L46.3 (GND), L47.1 (VDD), L47.3 (GND), L48.1 (VDD), L48.3 (GND), L5.1 (VDD), L5.3 (GND), L6.1 (VDD), L6.3 (GND), L7.1 (VDD), L7.3 (GND), L8.1 (VDD), L8.3 (GND), L9.1 (VDD), L9.3 (GND)
- net LED: now also L1.4 (DIN)
- new net: L33.2 (DOUT), L34.4 (DIN)
- new net: L32.2 (DOUT), L33.4 (DIN)
- new net: L24.2 (DOUT), L32.4 (DIN)
- new net: L24.4 (DIN), L25.2 (DOUT)
- new net: L13.4 (DIN), L14.2 (DOUT)
- new net: L14.4 (DIN), L15.2 (DOUT)
- new net: L29.4 (DIN), L30.2 (DOUT)
- new net: L30.4 (DIN), L31.2 (DOUT)
- new net: L15.4 (DIN), L7.2 (DOUT)
- new net: L6.2 (DOUT), L7.4 (DIN)
- new net: L17.2 (DOUT), L18.4 (DIN)
- new net: L16.2 (DOUT), L17.4 (DIN)
- new net: L10.2 (DOUT), L9.4 (DIN)
- new net: L10.4 (DIN), L11.2 (DOUT)
- new net: L1.2 (DOUT), L2.4 (DIN)
- new net: L43.4 (DIN), L44.2 (DOUT)
- new net: L44.4 (DIN), L45.2 (DOUT)
- new net: L40.4 (DIN), L41.2 (DOUT)
- new net: L41.4 (DIN), L42.2 (DOUT)
- new net: L45.4 (DIN), L46.2 (DOUT)
- new net: L27.4 (DIN), L28.2 (DOUT)
- new net: L28.4 (DIN), L29.2 (DOUT)
- new net: L4.2 (DOUT), L5.4 (DIN)
- new net: L3.2 (DOUT), L4.4 (DIN)
- new net: L39.2 (DOUT), L48.4 (DIN)
- new net: L38.2 (DOUT), L39.4 (DIN)
- new net: L47.4 (DIN), L48.2 (DOUT)
- new net: L26.4 (DIN), L27.2 (DOUT)
- new net: L42.4 (DIN), L43.2 (DOUT)
- new net: L11.4 (DIN), L12.2 (DOUT)
- new net: L21.2 (DOUT), L22.4 (DIN)
- new net: L20.2 (DOUT), L21.4 (DIN)
- new net: L23.2 (DOUT), L31.4 (DIN)
- new net: L8.4 (DIN), L9.2 (DOUT)
- new net: L37.2 (DOUT), L38.4 (DIN)
- new net: L5.2 (DOUT), L6.4 (DIN)
- new net: L16.4 (DIN), L8.2 (DOUT)
- new net: L35.2 (DOUT), L36.4 (DIN)
- new net: L34.2 (DOUT), L35.4 (DIN)
- new net: L25.4 (DIN), L26.2 (DOUT)
- new net: L2.2 (DOUT), L3.4 (DIN)
- new net: L18.2 (DOUT), L19.4 (DIN)
- new net: L36.2 (DOUT), L37.4 (DIN)
- new net: L46.4 (DIN), L47.2 (DOUT)
- new net: L12.4 (DIN), L13.2 (DOUT)
- new net: L22.2 (DOUT), L23.4 (DIN)
- no-connect marks 14 -> 17
Other:
- moved on the sheet: JP1, SW08_RH1B, SW10B, SW11B, SW12B, SW13B, SW14B, SW15B, SW16B, SW17B, SW18B, SW18_RH1B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

Commit message: Pico schematic switch nubmering changed to row/col intersection
Parts:
- removed D1, D10, D100, D101, D11, D12, D13, D14, D15, D16, D17, D18, D19, D2, D20, D21, D22, D23, D24, D25, D26, D27, D28, D29, D3, D30, D31, D32, D33, D34, D35, D36, D37, D38, D39, D4, D40, D41, D42, D43, D44, D45, D46, D47, D48, D49, D5, D50, D51, D52, D53, D54, D55, D56, D57, D58, D59, D6, D60, D61, D62, D63, D64, D65, D66, D67, D68, D69, D7, D70, D71, D72, D73, D74, D75, D76, D77, D78, D79, D8, D80, D81, D82, D83, D84, D85, D86, D87, D88, D89, D9, D90, D91, D92, D93, D94, D95, D96, D97, D98, D99: D, ergodonk_pico:D3_TH_SMD_v2, symbol Device:D
- removed JP1: LH LED's, Connector_PinHeader_2.54mm:PinHeader_1x02_P2.54mm_Vertical, symbol Jumper:SolderJumper_2_Open
- removed L1, L10, L11, L12, L13, L14, L15, L16, L17, L18, L19, L2, L20, L21, L22, L23, L24, L25, L26, L27, L28, L29, L3, L30, L31, L32, L33, L34, L35, L36, L37, L38, L39, L4, L40, L41, L42, L43, L44, L45, L46, L47, L48, L5, L6, L7, L8, L9: SK6812MINI-E, ergodonk_pico:SK6812-MINI-E, symbol Ergodonk_symbols:SK6812MINI
- removed SW08_RH1, SW10, SW11, SW15, SW18, SW18_RH1, SW19, SW20, SW21, SW24, SW25, SW27, SW28, SW28_RH1, SW31, SW33, SW35, SW36, SW38, SW38_RH1, SW40, SW41, SW42, SW45, SW48_RH1, SW5, SW6: SW_PUSH_LED, ergodonk_kicad_library:Chunky_2040_footprint_ergodonk_customs, symbol Ergodonk_symbols:SW_PUSH_LED
- removed SW1, SW100, SW101, SW12, SW13, SW14, SW16, SW17, SW2, SW22, SW23, SW26, SW29, SW3, SW30, SW32, SW34, SW37, SW39, SW4, SW43, SW44, SW46, SW47, SW48, SW49, SW50, SW51, SW52, SW53, SW54, SW55, SW56, SW57, SW58, SW59, SW60, SW61, SW62, SW63, SW64, SW65, SW66, SW67, SW68, SW69, SW7, SW70, SW71, SW72, SW73, SW74, SW75, SW76, SW77, SW78, SW79, SW8, SW80, SW81, SW82, SW83, SW84, SW86, SW87, SW88, SW89, SW9, SW90, SW91, SW92, SW93, SW94, SW95, SW96, SW97, SW98, SW99: SW_Push, symbol Switch:SW_Push
- added D_LH_00, D_LH_01, D_LH_02, D_LH_03, D_LH_04, D_LH_05, D_LH_06, D_LH_07, D_LH_10, D_LH_11, D_LH_12, D_LH_13, D_LH_14, D_LH_15, D_LH_16, D_LH_17, D_LH_20, D_LH_21, D_LH_22, D_LH_23, D_LH_24, D_LH_25, D_LH_26, D_LH_27, D_LH_30, D_LH_31, D_LH_32, D_LH_33, D_LH_34, D_LH_35, D_LH_36, D_LH_37, D_LH_40, D_LH_41, D_LH_42, D_LH_43, D_LH_44, D_LH_45, D_LH_46, D_LH_47, D_LH_50, D_LH_51, D_LH_52, D_LH_53, D_LH_54, D_LH_55, D_LH_56, D_LH_57, D_LH_58, D_RH_00, D_RH_01, D_RH_02, D_RH_03, D_RH_04, D_RH_05, D_RH_06, D_RH_07, D_RH_08, D_RH_10, D_RH_11, D_RH_12, D_RH_13, D_RH_14, D_RH_15, D_RH_16, D_RH_17, D_RH_18, D_RH_20, D_RH_21, D_RH_22, D_RH_23, D_RH_24, D_RH_25, D_RH_26, D_RH_27, D_RH_28, D_RH_30, D_RH_31, D_RH_32, D_RH_33, D_RH_34, D_RH_35, D_RH_36, D_RH_37, D_RH_38, D_RH_40, D_RH_41, D_RH_42, D_RH_43, D_RH_44, D_RH_45, D_RH_46, D_RH_47, D_RH_48, D_RH_50, D_RH_51, D_RH_52, D_RH_53, D_RH_54, D_RH_55, D_RH_56, D_RH_57, D_RH_58: D, symbol Device:D
- added SW_LH_00, SW_LH_01, SW_LH_02, SW_LH_03, SW_LH_04, SW_LH_05, SW_LH_06, SW_LH_07, SW_LH_10, SW_LH_11, SW_LH_12, SW_LH_13, SW_LH_14, SW_LH_15, SW_LH_16, SW_LH_17, SW_LH_20, SW_LH_21, SW_LH_22, SW_LH_23, SW_LH_24, SW_LH_25, SW_LH_26, SW_LH_27, SW_LH_30, SW_LH_31, SW_LH_32, SW_LH_33, SW_LH_34, SW_LH_35, SW_LH_36, SW_LH_37, SW_LH_40, SW_LH_42, SW_LH_43, SW_LH_44, SW_LH_45, SW_LH_46, SW_LH_47, SW_LH_50, SW_LH_51, SW_LH_52, SW_LH_53, SW_LH_54, SW_LH_55, SW_LH_56, SW_LH_57, SW_LH_58, SW_RH_00, SW_RH_01, SW_RH_02, SW_RH_03, SW_RH_04, SW_RH_05, SW_RH_06, SW_RH_07, SW_RH_08, SW_RH_10, SW_RH_11, SW_RH_12, SW_RH_13, SW_RH_14, SW_RH_15, SW_RH_16, SW_RH_17, SW_RH_18, SW_RH_20, SW_RH_21, SW_RH_22, SW_RH_23, SW_RH_24, SW_RH_25, SW_RH_26, SW_RH_27, SW_RH_28, SW_RH_30, SW_RH_31, SW_RH_32, SW_RH_33, SW_RH_34, SW_RH_35, SW_RH_36, SW_RH_37, SW_RH_38, SW_RH_40, SW_RH_42, SW_RH_43, SW_RH_44, SW_RH_45, SW_RH_46, SW_RH_47, SW_RH_48, SW_RH_50, SW_RH_51, SW_RH_52, SW_RH_53, SW_RH_54, SW_RH_55, SW_RH_56, SW_RH_57, SW_RH_58: SW_PUSH, symbol kbd:SW_PUSH
Connections:
- net GND: no longer D102.1 (K), D_SOL_1.C, J2.1 (Pin_1), J3.T, J_SOL_1.2 (Pin_2), OL1.3 (VCC), U2.39 (VSYS)
- net col0: now also SW_LH_00.1, SW_LH_10.1, SW_LH_20.1, SW_LH_30.1, SW_LH_40.1, SW_LH_50.1, SW_RH_00.1, SW_RH_10.1, SW_RH_20.1, SW_RH_30.1, SW_RH_40.1, SW_RH_50.1
- net col2: now also SW_LH_02.1, SW_LH_12.1, SW_LH_22.1, SW_LH_32.1, SW_LH_42.1, SW_LH_52.1, SW_RH_02.1, SW_RH_12.1, SW_RH_22.1, SW_RH_32.1, SW_RH_42.1, SW_RH_52.1
- net col3: now also SW_LH_03.1, SW_LH_13.1, SW_LH_23.1, SW_LH_33.1, SW_LH_43.1, SW_LH_53.1, SW_RH_03.1, SW_RH_13.1, SW_RH_23.1, SW_RH_33.1, SW_RH_43.1, SW_RH_53.1
- net col4: now also SW_LH_04.1, SW_LH_14.1, SW_LH_24.1, SW_LH_34.1, SW_LH_44.1, SW_LH_54.1, SW_RH_04.1, SW_RH_14.1, SW_RH_24.1, SW_RH_34.1, SW_RH_44.1, SW_RH_54.1
- net col5: now also SW_LH_05.1, SW_LH_15.1, SW_LH_25.1, SW_LH_35.1, SW_LH_45.1, SW_LH_55.1, SW_RH_05.1, SW_RH_15.1, SW_RH_25.1, SW_RH_35.1, SW_RH_45.1, SW_RH_55.1
- net col6: now also SW_LH_06.1, SW_LH_16.1, SW_LH_26.1, SW_LH_36.1, SW_LH_46.1, SW_LH_56.1, SW_RH_06.1, SW_RH_16.1, SW_RH_26.1, SW_RH_36.1, SW_RH_46.1, SW_RH_56.1
- net col7: now also SW_LH_07.1, SW_LH_17.1, SW_LH_27.1, SW_LH_37.1, SW_LH_47.1, SW_LH_57.1, SW_RH_07.1, SW_RH_17.1, SW_RH_27.1, SW_RH_37.1, SW_RH_47.1, SW_RH_57.1
- net col8: now also SW_LH_58.1, SW_RH_08.1, SW_RH_18.1, SW_RH_28.1, SW_RH_38.1, SW_RH_48.1, SW_RH_58.1
- net row0: now also D_LH_00.1 (K), D_LH_01.1 (K), D_LH_02.1 (K), D_LH_03.1 (K), D_LH_04.1 (K), D_LH_05.1 (K), D_LH_06.1 (K), D_LH_07.1 (K), D_RH_00.1 (K), D_RH_01.1 (K), D_RH_02.1 (K), D_RH_03.1 (K), D_RH_04.1 (K), D_RH_05.1 (K), D_RH_06.1 (K), D_RH_07.1 (K), D_RH_08.1 (K)
- net row1: now also D_LH_10.1 (K), D_LH_11.1 (K), D_LH_12.1 (K), D_LH_13.1 (K), D_LH_14.1 (K), D_LH_15.1 (K), D_LH_16.1 (K), D_LH_17.1 (K), D_RH_10.1 (K), D_RH_11.1 (K), D_RH_12.1 (K), D_RH_13.1 (K), D_RH_14.1 (K), D_RH_15.1 (K), D_RH_16.1 (K), D_RH_17.1 (K), D_RH_18.1 (K)
- net row2: now also D_LH_20.1 (K), D_LH_21.1 (K), D_LH_22.1 (K), D_LH_23.1 (K), D_LH_24.1 (K), D_LH_25.1 (K), D_LH_26.1 (K), D_LH_27.1 (K), D_RH_20.1 (K), D_RH_21.1 (K), D_RH_22.1 (K), D_RH_23.1 (K), D_RH_24.1 (K), D_RH_25.1 (K), D_RH_26.1 (K), D_RH_27.1 (K), D_RH_28.1 (K)
- net row3: now also D_LH_30.1 (K), D_LH_31.1 (K), D_LH_32.1 (K), D_LH_33.1 (K), D_LH_34.1 (K), D_LH_35.1 (K), D_LH_36.1 (K), D_LH_37.1 (K), D_RH_30.1 (K), D_RH_31.1 (K), D_RH_32.1 (K), D_RH_33.1 (K), D_RH_34.1 (K), D_RH_35.1 (K), D_RH_36.1 (K), D_RH_37.1 (K), D_RH_38.1 (K)
- net row4: now also D_LH_40.1 (K), D_LH_41.1 (K), D_LH_42.1 (K), D_LH_43.1 (K), D_LH_44.1 (K), D_LH_45.1 (K), D_LH_46.1 (K), D_LH_47.1 (K), D_RH_40.1 (K), D_RH_41.1 (K), D_RH_42.1 (K), D_RH_43.1 (K), D_RH_44.1 (K), D_RH_45.1 (K), D_RH_46.1 (K), D_RH_47.1 (K), D_RH_48.1 (K)
- net row5: now also D_LH_50.1 (K), D_LH_51.1 (K), D_LH_52.1 (K), D_LH_53.1 (K), D_LH_54.1 (K), D_LH_55.1 (K), D_LH_56.1 (K), D_LH_57.1 (K), D_LH_58.1 (K), D_RH_50.1 (K), D_RH_51.1 (K), D_RH_52.1 (K), D_RH_53.1 (K), D_RH_54.1 (K), D_RH_55.1 (K), D_RH_56.1 (K), D_RH_57.1 (K), D_RH_58.1 (K)
- net SW38_A renamed SW_LH_41_A
- net SW_LH_41_A: now also SW_LH_01.1, SW_LH_11.1, SW_LH_21.1, SW_LH_31.1, SW_LH_51.1, SW_RH_01.1, SW_RH_11.1, SW_RH_21.1, SW_RH_31.1, SW_RH_51.1
- net SW38_B renamed SW_LH_41_B
- net SW_LH_41_B: now also D_LH_41.2 (A)
- net SW85_B renamed SW_RH_41_B
- net SW_RH_41_B: now also D_RH_41.2 (A)
- new net: D_RH_17.2 (A), SW_RH_17.2
- new net: D_RH_35.2 (A), SW_RH_35.2
- new net: D_LH_35.2 (A), SW_LH_35.2
- new net: D_LH_43.2 (A), SW_LH_43.2
- new net: D_LH_01.2 (A), SW_LH_01.2
- new net: D_LH_25.2 (A), SW_LH_25.2
- new net: D_LH_23.2 (A), SW_LH_23.2
- new net: D_LH_24.2 (A), SW_LH_24.2
- new net: D_LH_20.2 (A), SW_LH_20.2
- new net: D_RH_03.2 (A), SW_RH_03.2
- new net: D_LH_54.2 (A), SW_LH_54.2
- new net: D_RH_04.2 (A), SW_RH_04.2
- new net: D_LH_36.2 (A), SW_LH_36.2
- new net: D_RH_27.2 (A), SW_RH_27.2
- new net: D_LH_56.2 (A), SW_LH_56.2
- new net: D_RH_26.2 (A), SW_RH_26.2
- new net: D_LH_14.2 (A), SW_LH_14.2
- new net: D_RH_48.2 (A), SW_RH_48.2
- new net: D_LH_02.2 (A), SW_LH_02.2
- new net: D_RH_10.2 (A), SW_RH_10.2
- new net: D_RH_30.2 (A), SW_RH_30.2
- new net: D_RH_55.2 (A), SW_RH_55.2
- new net: D_RH_46.2 (A), SW_RH_46.2
- new net: D_LH_06.2 (A), SW_LH_06.2
- new net: D_RH_37.2 (A), SW_RH_37.2
- new net: D_RH_51.2 (A), SW_RH_51.2
- new net: D_LH_55.2 (A), SW_LH_55.2
- new net: D_RH_31.2 (A), SW_RH_31.2
- new net: D_RH_13.2 (A), SW_RH_13.2
- new net: D_RH_22.2 (A), SW_RH_22.2
- new net: D_RH_52.2 (A), SW_RH_52.2
- new net: D_LH_34.2 (A), SW_LH_34.2
- new net: D_RH_54.2 (A), SW_RH_54.2
- new net: D_RH_11.2 (A), SW_RH_11.2
- new net: D_LH_47.2 (A), SW_LH_47.2
- new net: D_RH_25.2 (A), SW_RH_25.2
- new net: D_RH_42.2 (A), SW_RH_42.2
- new net: D_RH_15.2 (A), SW_RH_15.2
- new net: D_LH_45.2 (A), SW_LH_45.2
- new net: D_LH_05.2 (A), SW_LH_05.2
- new net: D_LH_12.2 (A), SW_LH_12.2
- new net: D_LH_46.2 (A), SW_LH_46.2
- new net: D_LH_07.2 (A), SW_LH_07.2
- new net: D_LH_58.2 (A), SW_LH_58.2
- new net: D_LH_26.2 (A), SW_LH_26.2
- new net: D_RH_01.2 (A), SW_RH_01.2
- new net: D_RH_18.2 (A), SW_RH_18.2
- new net: D_RH_06.2 (A), SW_RH_06.2
- new net: D_RH_08.2 (A), SW_RH_08.2
- new net: D_LH_22.2 (A), SW_LH_22.2
- new net: D_RH_32.2 (A), SW_RH_32.2
- new net: D_LH_03.2 (A), SW_LH_03.2
- new net: D_LH_53.2 (A), SW_LH_53.2
- new net: D_RH_34.2 (A), SW_RH_34.2
- new net: D_LH_11.2 (A), SW_LH_11.2
- new net: D_RH_53.2 (A), SW_RH_53.2
- new net: D_LH_16.2 (A), SW_LH_16.2
- new net: D_LH_27.2 (A), SW_LH_27.2
- new net: D_RH_28.2 (A), SW_RH_28.2
- new net: D_RH_05.2 (A), SW_RH_05.2
- new net: D_LH_17.2 (A), SW_LH_17.2
- new net: D_LH_00.2 (A), SW_LH_00.2
- new net: D_RH_20.2 (A), SW_RH_20.2
- new net: D_RH_43.2 (A), SW_RH_43.2
- new net: D_LH_21.2 (A), SW_LH_21.2
- new net: D_LH_32.2 (A), SW_LH_32.2
- new net: D_LH_50.2 (A), SW_LH_50.2
- new net: D_RH_12.2 (A), SW_RH_12.2
- new net: D_LH_57.2 (A), SW_LH_57.2
- new net: D_RH_56.2 (A), SW_RH_56.2
- new net: D_RH_40.2 (A), SW_RH_40.2
- new net: D_RH_44.2 (A), SW_RH_44.2
- new net: D_RH_45.2 (A), SW_RH_45.2
- new net: D_RH_38.2 (A), SW_RH_38.2
- new net: D_LH_13.2 (A), SW_LH_13.2
- new net: D_LH_33.2 (A), SW_LH_33.2
- new net: D_LH_15.2 (A), SW_LH_15.2
- new net: D_LH_52.2 (A), SW_LH_52.2
- new net: D_RH_14.2 (A), SW_RH_14.2
- new net: D_RH_57.2 (A), SW_RH_57.2
- new net: D_RH_02.2 (A), SW_RH_02.2
- new net: D_RH_16.2 (A), SW_RH_16.2
- new net: D_LH_37.2 (A), SW_LH_37.2
- new net: D_RH_07.2 (A), SW_RH_07.2
- new net: D_LH_42.2 (A), SW_LH_42.2
- new net: D_RH_23.2 (A), SW_RH_23.2
- new net: D_RH_00.2 (A), SW_RH_00.2
- new net: D_RH_36.2 (A), SW_RH_36.2
- new net: D_LH_51.2 (A), SW_LH_51.2
- new net: D_RH_50.2 (A), SW_RH_50.2
- new net: D_LH_31.2 (A), SW_LH_31.2
- new net: D_LH_10.2 (A), SW_LH_10.2
- new net: D_RH_21.2 (A), SW_RH_21.2
- new net: D_LH_40.2 (A), SW_LH_40.2
- new net: D_RH_58.2 (A), SW_RH_58.2
- new net: D_RH_47.2 (A), SW_RH_47.2
- new net: D_LH_30.2 (A), SW_LH_30.2
- new net: D_RH_33.2 (A), SW_RH_33.2
- new net: D_LH_04.2 (A), SW_LH_04.2
- new net: D_RH_24.2 (A), SW_RH_24.2
- new net: D_LH_44.2 (A), SW_LH_44.2
- new net VCC: D102.1 (K), D_SOL_1.C, J2.1 (Pin_1), J3.T, J_SOL_1.2 (Pin_2), OL1.3 (VCC), U2.39 (VSYS)
- no-connect marks 17 -> 13
Other:
- note added: "Note: Switches are numbered according to row/column intersection."
- note removed: "@TODO: Do we want a new footprint for rotary encoder/switch with LED?"
- note removed: "Alpha Keys (LH & RH)"
- note removed: "Aux Keys"
- note removed: "F keys"
- note removed: "LED's 1) Based on Keebio Sync rev3, we can put in all these LED's if we limit brightness Add a jumper if you want to make the LH snap off for assymetry."
- note removed: "RH Only"
- note removed: "Rotary Encoder"
- note removed: "Thumb Cluster"

Commit message: Pico leds re-added to schemematic PCB rough key layout
Parts:
- added L_LH_00, L_LH_1, L_LH_10, L_LH_11, L_LH_12, L_LH_13, L_LH_14, L_LH_15, L_LH_16, L_LH_17, L_LH_2, L_LH_20, L_LH_21, L_LH_22, L_LH_23, L_LH_24, L_LH_25, L_LH_26, L_LH_27, L_LH_3, L_LH_30, L_LH_31, L_LH_32, L_LH_33, L_LH_34, L_LH_35, L_LH_36, L_LH_37, L_LH_4, L_LH_40, L_LH_41, L_LH_42, L_LH_43, L_LH_44, L_LH_45, L_LH_46, L_LH_47, L_LH_5, L_LH_50, L_LH_51, L_LH_52, L_LH_53, L_LH_54, L_LH_55, L_LH_56, L_LH_57, L_LH_58, L_LH_6, L_LH_7, L_RH_00, L_RH_1, L_RH_10, L_RH_11, L_RH_12, L_RH_13, L_RH_14, L_RH_15, L_RH_16, L_RH_17, L_RH_18, L_RH_2, L_RH_20, L_RH_21, L_RH_22, L_RH_23, L_RH_24, L_RH_25, L_RH_26, L_RH_27, L_RH_28, L_RH_3, L_RH_30, L_RH_31, L_RH_32, L_RH_33, L_RH_34, L_RH_35, L_RH_36, L_RH_37, L_RH_38, L_RH_4, L_RH_40, L_RH_41, L_RH_42, L_RH_43, L_RH_44, L_RH_45, L_RH_46, L_RH_47, L_RH_48, L_RH_5, L_RH_50, L_RH_51, L_RH_52, L_RH_53, L_RH_54, L_RH_55, L_RH_56, L_RH_57, L_RH_58, L_RH_6, L_RH_7, L_RH_8: SK6812MINI-E, ergodonk_pico:SK6812-MINI-E, symbol Ergodonk_symbols:SK6812MINI
- D_LH_00, D_LH_01, D_LH_02, D_LH_03, D_LH_04, D_LH_05, D_LH_06, D_LH_07, D_LH_10, D_LH_11, D_LH_12, D_LH_13, D_LH_14, D_LH_15, D_LH_16, D_LH_17, D_LH_20, D_LH_21, D_LH_22, D_LH_23, D_LH_24, D_LH_25, D_LH_26, D_LH_27, D_LH_30, D_LH_31, D_LH_32, D_LH_33, D_LH_34, D_LH_35, D_LH_36, D_LH_37, D_LH_40, D_LH_41, D_LH_42, D_LH_43, D_LH_44, D_LH_45, D_LH_46, D_LH_47, D_LH_50, D_LH_51, D_LH_52, D_LH_53, D_LH_54, D_LH_55, D_LH_56, D_LH_57, D_LH_58, D_RH_00, D_RH_01, D_RH_02, D_RH_03, D_RH_04, D_RH_05, D_RH_06, D_RH_07, D_RH_08, D_RH_10, D_RH_11, D_RH_12, D_RH_13, D_RH_14, D_RH_15, D_RH_16, D_RH_17, D_RH_18, D_RH_20, D_RH_21, D_RH_22, D_RH_23, D_RH_24, D_RH_25, D_RH_26, D_RH_27, D_RH_28, D_RH_30, D_RH_31, D_RH_32, D_RH_33, D_RH_34, D_RH_35, D_RH_36, D_RH_37, D_RH_38, D_RH_40, D_RH_41, D_RH_42, D_RH_43, D_RH_44, D_RH_45, D_RH_46, D_RH_47, D_RH_48, D_RH_50, D_RH_51, D_RH_52, D_RH_53, D_RH_54, D_RH_55, D_RH_56, D_RH_57, D_RH_58: footprint (none) -> ergodonk_pico:D3_TH_SMD_v2
- SW_LH_00, SW_LH_01, SW_LH_02, SW_LH_03, SW_LH_04, SW_LH_05, SW_LH_06, SW_LH_07, SW_LH_10, SW_LH_11, SW_LH_12, SW_LH_13, SW_LH_14, SW_LH_15, SW_LH_16, SW_LH_17, SW_LH_20, SW_LH_21, SW_LH_22, SW_LH_23, SW_LH_24, SW_LH_25, SW_LH_26, SW_LH_27, SW_LH_30, SW_LH_31, SW_LH_32, SW_LH_33, SW_LH_34, SW_LH_35, SW_LH_36, SW_LH_37, SW_LH_40, SW_LH_42, SW_LH_43, SW_LH_44, SW_LH_45, SW_LH_46, SW_LH_47, SW_LH_50, SW_LH_51, SW_LH_52, SW_LH_53, SW_LH_54, SW_LH_55, SW_LH_56, SW_LH_57, SW_LH_58, SW_RH_00, SW_RH_01, SW_RH_02, SW_RH_03, SW_RH_04, SW_RH_05, SW_RH_06, SW_RH_07, SW_RH_08, SW_RH_10, SW_RH_11, SW_RH_12, SW_RH_13, SW_RH_14, SW_RH_15, SW_RH_16, SW_RH_17, SW_RH_18, SW_RH_20, SW_RH_21, SW_RH_22, SW_RH_23, SW_RH_24, SW_RH_25, SW_RH_26, SW_RH_27, SW_RH_28, SW_RH_30, SW_RH_31, SW_RH_32, SW_RH_33, SW_RH_34, SW_RH_35, SW_RH_36, SW_RH_37, SW_RH_38, SW_RH_40, SW_RH_42, SW_RH_43, SW_RH_44, SW_RH_45, SW_RH_46, SW_RH_47, SW_RH_48, SW_RH_50, SW_RH_51, SW_RH_52, SW_RH_53, SW_RH_54, SW_RH_55, SW_RH_56, SW_RH_57, SW_RH_58: footprint (none) -> ergodonk_pico:Chunky_2040_footprint_ergodonk_customs
Connections:
- net GND: now also L_LH_00.3 (GND), L_LH_1.3 (GND), L_LH_10.3 (GND), L_LH_11.3 (GND), L_LH_12.3 (GND), L_LH_13.3 (GND), L_LH_14.3 (GND), L_LH_15.3 (GND), L_LH_16.3 (GND), L_LH_17.3 (GND), L_LH_2.3 (GND), L_LH_20.3 (GND), L_LH_21.3 (GND), L_LH_22.3 (GND), L_LH_23.3 (GND), L_LH_24.3 (GND), L_LH_25.3 (GND), L_LH_26.3 (GND), L_LH_27.3 (GND), L_LH_3.3 (GND), L_LH_30.3 (GND), L_LH_31.3 (GND), L_LH_32.3 (GND), L_LH_33.3 (GND), L_LH_34.3 (GND), L_LH_35.3 (GND), L_LH_36.3 (GND), L_LH_37.3 (GND), L_LH_4.3 (GND), L_LH_40.3 (GND), L_LH_41.3 (GND), L_LH_42.3 (GND), L_LH_43.3 (GND), L_LH_44.3 (GND), L_LH_45.3 (GND), L_LH_46.3 (GND), L_LH_47.3 (GND), L_LH_5.3 (GND), L_LH_50.3 (GND), L_LH_51.3 (GND), L_LH_52.3 (GND), L_LH_53.3 (GND), L_LH_54.3 (GND), L_LH_55.3 (GND), L_LH_56.3 (GND), L_LH_57.3 (GND), L_LH_58.3 (GND), L_LH_6.3 (GND), L_LH_7.3 (GND), L_RH_00.3 (GND), L_RH_1.3 (GND), L_RH_10.3 (GND), L_RH_11.3 (GND), L_RH_12.3 (GND), L_RH_13.3 (GND), L_RH_14.3 (GND), L_RH_15.3 (GND), L_RH_16.3 (GND), L_RH_17.3 (GND), L_RH_18.3 (GND), L_RH_2.3 (GND), L_RH_20.3 (GND), L_RH_21.3 (GND), L_RH_22.3 (GND), L_RH_23.3 (GND), L_RH_24.3 (GND), L_RH_25.3 (GND), L_RH_26.3 (GND), L_RH_27.3 (GND), L_RH_28.3 (GND), L_RH_3.3 (GND), L_RH_30.3 (GND), L_RH_31.3 (GND), L_RH_32.3 (GND), L_RH_33.3 (GND), L_RH_34.3 (GND), L_RH_35.3 (GND), L_RH_36.3 (GND), L_RH_37.3 (GND), L_RH_38.3 (GND), L_RH_4.3 (GND), L_RH_40.3 (GND), L_RH_41.3 (GND), L_RH_42.3 (GND), L_RH_43.3 (GND), L_RH_44.3 (GND), L_RH_45.3 (GND), L_RH_46.3 (GND), L_RH_47.3 (GND), L_RH_48.3 (GND), L_RH_5.3 (GND), L_RH_50.3 (GND), L_RH_51.3 (GND), L_RH_52.3 (GND), L_RH_53.3 (GND), L_RH_54.3 (GND), L_RH_55.3 (GND), L_RH_56.3 (GND), L_RH_57.3 (GND), L_RH_58.3 (GND), L_RH_6.3 (GND), L_RH_7.3 (GND), L_RH_8.3 (GND)
- new net VDD: L_LH_00.1 (VDD), L_LH_1.1 (VDD), L_LH_10.1 (VDD), L_LH_11.1 (VDD), L_LH_12.1 (VDD), L_LH_13.1 (VDD), L_LH_14.1 (VDD), L_LH_15.1 (VDD), L_LH_16.1 (VDD), L_LH_17.1 (VDD), L_LH_2.1 (VDD), L_LH_20.1 (VDD), L_LH_21.1 (VDD), L_LH_22.1 (VDD), L_LH_23.1 (VDD), L_LH_24.1 (VDD), L_LH_25.1 (VDD), L_LH_26.1 (VDD), L_LH_27.1 (VDD), L_LH_3.1 (VDD), L_LH_30.1 (VDD), L_LH_31.1 (VDD), L_LH_32.1 (VDD), L_LH_33.1 (VDD), L_LH_34.1 (VDD), L_LH_35.1 (VDD), L_LH_36.1 (VDD), L_LH_37.1 (VDD), L_LH_4.1 (VDD), L_LH_40.1 (VDD), L_LH_41.1 (VDD), L_LH_42.1 (VDD), L_LH_43.1 (VDD), L_LH_44.1 (VDD), L_LH_45.1 (VDD), L_LH_46.1 (VDD), L_LH_47.1 (VDD), L_LH_5.1 (VDD), L_LH_50.1 (VDD), L_LH_51.1 (VDD), L_LH_52.1 (VDD), L_LH_53.1 (VDD), L_LH_54.1 (VDD), L_LH_55.1 (VDD), L_LH_56.1 (VDD), L_LH_57.1 (VDD), L_LH_58.1 (VDD), L_LH_6.1 (VDD), L_LH_7.1 (VDD), L_RH_00.1 (VDD), L_RH_1.1 (VDD), L_RH_10.1 (VDD), L_RH_11.1 (VDD), L_RH_12.1 (VDD), L_RH_13.1 (VDD), L_RH_14.1 (VDD), L_RH_15.1 (VDD), L_RH_16.1 (VDD), L_RH_17.1 (VDD), L_RH_18.1 (VDD), L_RH_2.1 (VDD), L_RH_20.1 (VDD), L_RH_21.1 (VDD), L_RH_22.1 (VDD), L_RH_23.1 (VDD), L_RH_24.1 (VDD), L_RH_25.1 (VDD), L_RH_26.1 (VDD), L_RH_27.1 (VDD), L_RH_28.1 (VDD), L_RH_3.1 (VDD), L_RH_30.1 (VDD), L_RH_31.1 (VDD), L_RH_32.1 (VDD), L_RH_33.1 (VDD), L_RH_34.1 (VDD), L_RH_35.1 (VDD), L_RH_36.1 (VDD), L_RH_37.1 (VDD), L_RH_38.1 (VDD), L_RH_4.1 (VDD), L_RH_40.1 (VDD), L_RH_41.1 (VDD), L_RH_42.1 (VDD), L_RH_43.1 (VDD), L_RH_44.1 (VDD), L_RH_45.1 (VDD), L_RH_46.1 (VDD), L_RH_47.1 (VDD), L_RH_48.1 (VDD), L_RH_5.1 (VDD), L_RH_50.1 (VDD), L_RH_51.1 (VDD), L_RH_52.1 (VDD), L_RH_53.1 (VDD), L_RH_54.1 (VDD), L_RH_55.1 (VDD), L_RH_56.1 (VDD), L_RH_57.1 (VDD), L_RH_58.1 (VDD), L_RH_6.1 (VDD), L_RH_7.1 (VDD), L_RH_8.1 (VDD)
Other:
- moved on the sheet: S1
