File: ergodonk_pico/ergodonk_pico.kicad_sch (KiCad schematic)
At the start: 333 parts, among them J2 Pimaroni Trackball, J3 AudioJack4, Q1 TIP120, U2 Pico

Commit message: Revised RH row/columns for syntactic sugar
Parts:
- removed SW_RH_32: SW_PUSH, ergodonk_pico:Chunky_2040_footprint_ergodonk_customs, symbol kbd:SW_PUSH
- L_LH_00, L_LH_1, L_LH_10, L_LH_11, L_LH_12, L_LH_13, L_LH_14, L_LH_15, L_LH_16, L_LH_17, L_LH_2, L_LH_20, L_LH_21, L_LH_22, L_LH_23, L_LH_24, L_LH_25, L_LH_26, L_LH_27, L_LH_3, L_LH_30, L_LH_31, L_LH_32, L_LH_33, L_LH_34, L_LH_35, L_LH_36, L_LH_37, L_LH_4, L_LH_40, L_LH_41, L_LH_42, L_LH_43, L_LH_44, L_LH_45, L_LH_46, L_LH_47, L_LH_5, L_LH_50, L_LH_51, L_LH_52, L_LH_53, L_LH_54, L_LH_55, L_LH_56, L_LH_57, L_LH_58, L_LH_6, L_LH_7, L_RH_00, L_RH_1, L_RH_10, L_RH_11, L_RH_12, L_RH_13, L_RH_14, L_RH_15, L_RH_16, L_RH_17, L_RH_18, L_RH_2, L_RH_20, L_RH_21, L_RH_22, L_RH_23, L_RH_24, L_RH_25, L_RH_26, L_RH_27, L_RH_28, L_RH_3, L_RH_30, L_RH_31, L_RH_32, L_RH_33, L_RH_34, L_RH_35, L_RH_36, L_RH_37, L_RH_38, L_RH_4, L_RH_40, L_RH_41, L_RH_42, L_RH_43, L_RH_44, L_RH_45, L_RH_46, L_RH_47, L_RH_48, L_RH_5, L_RH_50, L_RH_51, L_RH_52, L_RH_53, L_RH_54, L_RH_55, L_RH_56, L_RH_57, L_RH_58, L_RH_6, L_RH_7, L_RH_8: footprint ergodonk_pico:SK6812-MINI-E -> ergodonk_pico:V2_CherryMX_Hotswap
- SW_LH_00, SW_LH_01, SW_LH_02, SW_LH_03, SW_LH_04, SW_LH_05, SW_LH_06, SW_LH_07, SW_LH_10, SW_LH_11, SW_LH_12, SW_LH_13, SW_LH_14, SW_LH_15, SW_LH_16, SW_LH_17, SW_LH_20, SW_LH_21, SW_LH_22, SW_LH_23, SW_LH_24, SW_LH_25, SW_LH_26, SW_LH_27, SW_LH_30, SW_LH_31, SW_LH_32, SW_LH_33, SW_LH_34, SW_LH_35, SW_LH_36, SW_LH_37, SW_LH_40, SW_LH_42, SW_LH_43, SW_LH_44, SW_LH_45, SW_LH_46, SW_LH_47, SW_LH_50, SW_LH_53, SW_LH_54, SW_LH_55, SW_LH_56, SW_LH_57, SW_LH_58, SW_RH_00, SW_RH_01, SW_RH_02, SW_RH_03, SW_RH_04, SW_RH_05, SW_RH_06, SW_RH_07, SW_RH_08, SW_RH_10, SW_RH_11, SW_RH_12, SW_RH_13, SW_RH_14, SW_RH_15, SW_RH_16, SW_RH_17, SW_RH_18, SW_RH_20, SW_RH_21, SW_RH_22, SW_RH_23, SW_RH_24, SW_RH_25, SW_RH_26, SW_RH_27, SW_RH_28, SW_RH_30, SW_RH_31, SW_RH_33, SW_RH_34, SW_RH_35, SW_RH_36, SW_RH_37, SW_RH_38, SW_RH_40, SW_RH_42, SW_RH_43, SW_RH_44, SW_RH_45, SW_RH_46, SW_RH_47, SW_RH_48, SW_RH_50, SW_RH_51, SW_RH_52, SW_RH_53, SW_RH_54, SW_RH_55, SW_RH_56, SW_RH_57, SW_RH_58: footprint ergodonk_pico:Chunky_2040_footprint_ergodonk_customs -> ergodonk_pico:V2_CherryMX_Hotswap
- SW_LH_51, SW_LH_52: footprint ergodonk_pico:Chunky_2040_footprint_ergodonk_customs -> ergodonk_pico:V2_CherryMX_KailhV2_Hotswap
- U2: footprint ergodonk_kicad_library:RPi_Pico_SMD_TH -> ergodonk_pico:RPi_Pico_SMD_TH_DS_Ergodonk_v1
Connections:
- net SW_LH_41_A: no longer SWRH_ROT1.S1, SW_RH_01.1, SW_RH_11.1, SW_RH_21.1, SW_RH_31.1, SW_RH_51.1
- net col0: no longer SW_RH_00.1, SW_RH_10.1, SW_RH_20.1, SW_RH_30.1, SW_RH_40.1, SW_RH_50.1
- net col2: no longer SW_RH_02.1, SW_RH_12.1, SW_RH_22.1, SW_RH_42.1, SW_RH_52.1
- net col3: no longer SW_RH_03.1, SW_RH_13.1, SW_RH_23.1, SW_RH_33.1, SW_RH_43.1, SW_RH_53.1
- net col4: no longer SW_RH_04.1, SW_RH_14.1, SW_RH_24.1, SW_RH_34.1, SW_RH_44.1, SW_RH_54.1
- net col5: no longer SW_RH_05.1, SW_RH_15.1, SW_RH_25.1, SW_RH_35.1, SW_RH_45.1, SW_RH_55.1
- net col6: no longer SW_RH_06.1, SW_RH_16.1, SW_RH_26.1, SW_RH_36.1, SW_RH_46.1, SW_RH_56.1
- net col7: no longer SW_RH_07.1, SW_RH_17.1, SW_RH_27.1, SW_RH_37.1, SW_RH_47.1, SW_RH_57.1
- net col8: no longer SW_RH_08.1, SW_RH_18.1, SW_RH_28.1, SW_RH_38.1, SW_RH_48.1, SW_RH_58.1
- net row0: no longer D_RH_00.1 (K), D_RH_01.1 (K), D_RH_02.1 (K), D_RH_03.1 (K), D_RH_04.1 (K), D_RH_05.1 (K), D_RH_06.1 (K), D_RH_07.1 (K), D_RH_08.1 (K)
- net row1: no longer D_RH_10.1 (K), D_RH_11.1 (K), D_RH_12.1 (K), D_RH_13.1 (K), D_RH_14.1 (K), D_RH_15.1 (K), D_RH_16.1 (K), D_RH_17.1 (K), D_RH_18.1 (K)
- net row2: no longer D_RH_20.1 (K), D_RH_21.1 (K), D_RH_22.1 (K), D_RH_23.1 (K), D_RH_24.1 (K), D_RH_25.1 (K), D_RH_26.1 (K), D_RH_27.1 (K), D_RH_28.1 (K)
- net row3: no longer D_RH_30.1 (K), D_RH_31.1 (K), D_RH_32.1 (K), D_RH_33.1 (K), D_RH_34.1 (K), D_RH_35.1 (K), D_RH_36.1 (K), D_RH_37.1 (K), D_RH_38.1 (K)
- net row4: no longer D_RH_40.1 (K), D_RH_41.1 (K), D_RH_42.1 (K), D_RH_43.1 (K), D_RH_44.1 (K), D_RH_45.1 (K), D_RH_46.1 (K), D_RH_47.1 (K), D_RH_48.1 (K)
- net row5: no longer D_RH_50.1 (K), D_RH_51.1 (K), D_RH_52.1 (K), D_RH_53.1 (K), D_RH_54.1 (K), D_RH_55.1 (K), D_RH_56.1 (K), D_RH_57.1 (K), D_RH_58.1 (K)
- new net SW_RH_41_A: SWRH_ROT1.S1, SW_RH_01.1, SW_RH_11.1, SW_RH_21.1, SW_RH_31.1, SW_RH_51.1
- new net col0_rh: SW_RH_00.1, SW_RH_10.1, SW_RH_20.1, SW_RH_30.1, SW_RH_40.1, SW_RH_50.1
- new net col2_rh: SW_RH_02.1, SW_RH_12.1, SW_RH_22.1, SW_RH_42.1, SW_RH_52.1
- new net col3_rh: SW_RH_03.1, SW_RH_13.1, SW_RH_23.1, SW_RH_33.1, SW_RH_43.1, SW_RH_53.1
- new net col4_rh: SW_RH_04.1, SW_RH_14.1, SW_RH_24.1, SW_RH_34.1, SW_RH_44.1, SW_RH_54.1
- new net col5_rh: SW_RH_05.1, SW_RH_15.1, SW_RH_25.1, SW_RH_35.1, SW_RH_45.1, SW_RH_55.1
- new net col6_rh: SW_RH_06.1, SW_RH_16.1, SW_RH_26.1, SW_RH_36.1, SW_RH_46.1, SW_RH_56.1
- new net col7_rh: SW_RH_07.1, SW_RH_17.1, SW_RH_27.1, SW_RH_37.1, SW_RH_47.1, SW_RH_57.1
- new net col8_rh: SW_RH_08.1, SW_RH_18.1, SW_RH_28.1, SW_RH_38.1, SW_RH_48.1, SW_RH_58.1
- new net row0_rh: D_RH_00.1 (K), D_RH_01.1 (K), D_RH_02.1 (K), D_RH_03.1 (K), D_RH_04.1 (K), D_RH_05.1 (K), D_RH_06.1 (K), D_RH_07.1 (K), D_RH_08.1 (K)
- new net row1_rh: D_RH_10.1 (K), D_RH_11.1 (K), D_RH_12.1 (K), D_RH_13.1 (K), D_RH_14.1 (K), D_RH_15.1 (K), D_RH_16.1 (K), D_RH_17.1 (K), D_RH_18.1 (K)
- new net row2_rh: D_RH_20.1 (K), D_RH_21.1 (K), D_RH_22.1 (K), D_RH_23.1 (K), D_RH_24.1 (K), D_RH_25.1 (K), D_RH_26.1 (K), D_RH_27.1 (K), D_RH_28.1 (K)
- new net row3_rh: D_RH_30.1 (K), D_RH_31.1 (K), D_RH_32.1 (K), D_RH_33.1 (K), D_RH_34.1 (K), D_RH_35.1 (K), D_RH_36.1 (K), D_RH_37.1 (K), D_RH_38.1 (K)
- new net row4_rh: D_RH_40.1 (K), D_RH_41.1 (K), D_RH_42.1 (K), D_RH_43.1 (K), D_RH_44.1 (K), D_RH_45.1 (K), D_RH_46.1 (K), D_RH_47.1 (K), D_RH_48.1 (K)
- new net row5_rh: D_RH_50.1 (K), D_RH_51.1 (K), D_RH_52.1 (K), D_RH_53.1 (K), D_RH_54.1 (K), D_RH_55.1 (K), D_RH_56.1 (K), D_RH_57.1 (K), D_RH_58.1 (K)

Commit message: Thumb rotation diode placement added tenting puck symbols and footprint
Parts:
- added H14, H15: Tenting puck mount, ergodonk_kicad_library:Tenting_Puck.kicad_mod_nocenter, symbol Mechanical:MountingHole
- added SW_RH_32: SW_PUSH, ergodonk_pico:V2_CherryMX_Hotswap, symbol kbd:SW_PUSH
- L_LH_00, L_LH_1, L_LH_10, L_LH_11, L_LH_12, L_LH_13, L_LH_14, L_LH_15, L_LH_16, L_LH_17, L_LH_2, L_LH_20, L_LH_21, L_LH_22, L_LH_23, L_LH_24, L_LH_25, L_LH_26, L_LH_27, L_LH_3, L_LH_30, L_LH_31, L_LH_32, L_LH_33, L_LH_34, L_LH_35, L_LH_36, L_LH_37, L_LH_4, L_LH_40, L_LH_41, L_LH_42, L_LH_43, L_LH_44, L_LH_45, L_LH_46, L_LH_47, L_LH_5, L_LH_50, L_LH_51, L_LH_52, L_LH_53, L_LH_54, L_LH_55, L_LH_56, L_LH_57, L_LH_58, L_LH_6, L_LH_7, L_RH_00, L_RH_1, L_RH_10, L_RH_11, L_RH_12, L_RH_13, L_RH_14, L_RH_15, L_RH_16, L_RH_17, L_RH_18, L_RH_2, L_RH_20, L_RH_21, L_RH_22, L_RH_23, L_RH_24, L_RH_25, L_RH_26, L_RH_27, L_RH_28, L_RH_3, L_RH_30, L_RH_31, L_RH_32, L_RH_33, L_RH_34, L_RH_35, L_RH_36, L_RH_37, L_RH_38, L_RH_4, L_RH_40, L_RH_41, L_RH_42, L_RH_43, L_RH_44, L_RH_45, L_RH_46, L_RH_47, L_RH_48, L_RH_5, L_RH_50, L_RH_51, L_RH_52, L_RH_53, L_RH_54, L_RH_55, L_RH_56, L_RH_57, L_RH_58, L_RH_6, L_RH_7, L_RH_8: footprint ergodonk_pico:V2_CherryMX_Hotswap -> ergodonk_pico:SK6812-MINI-E
- SW_RH_51, SW_RH_52: footprint ergodonk_pico:V2_CherryMX_Hotswap -> ergodonk_pico:V2_CherryMX_KailhV2_Hotswap
Connections:
- net col2_rh: now also SW_RH_32.1
- net at D_RH_32.2 (A): now also SW_RH_32.2

Commit message: Added pmw3360 schematic for pico
Parts:
- removed J2: Pimaroni Trackball, ergodonk_kicad_library:pimoroni_trackball, symbol Connector:Conn_01x05_Socket
- removed J3: AudioJack4, ergodonk_kicad_library:MJ-4PP-9_CANTOR_KITCHEN_SINK, symbol Connector:AudioJack4
- added D1: D, ergodonk_pico:D3_TH_SMD_v2, symbol Device:D
- added J1, J4: AudioJack4, ergodonk_kicad_library:MJ-4PP-9_CANTOR_KITCHEN_SINK, symbol Connector:AudioJack4
- added J2: Conn_01x08_Socket, symbol Connector:Conn_01x08_Socket
- added U2: Pico, ergodonk_pico:RPi_Pico_SMD_TH_DS_Ergodonk_v1, symbol Pico:Pico
- renumbered U2 to U1
Connections:
- net GND: now also J1.S, J2.2 (Pin_2), J4.S, U2.13 (GND), U2.18 (GND), U2.23 (GND), U2.28 (GND), U2.3 (GND), U2.33 (AGND), U2.38 (GND), U2.8 (GND)
- net LED: now also U1.20 (GPIO15), U2.20 (GPIO15); no longer U1.25 (GPIO19)
- net SCL: now also U1.32 (GPIO27_ADC1), U2.32 (GPIO27_ADC1); no longer U1.27 (GPIO21)
- net SDA: now also U1.31 (GPIO26_ADC0), U2.31 (GPIO26_ADC0); no longer U1.26 (GPIO20)
- net SOLENOID_CONTROL: now also U1.26 (GPIO20); no longer U1.29 (GPIO22)
- net SPEAKER: now also U1.27 (GPIO21); no longer U1.31 (GPIO26_ADC0)
- net SW_LH_41_A: now also U2.12 (GPIO9)
- net VCC: now also D1.1 (K), J1.T, J4.T, U2.39 (VSYS)
- net col0: now also U2.11 (GPIO8)
- net col2: now also U2.14 (GPIO10)
- net col3: now also U2.15 (GPIO11)
- net col4: now also U2.16 (GPIO12)
- net col5: now also U2.17 (GPIO13)
- net col6: now also U2.19 (GPIO14)
- net col7: now also U1.34 (GPIO28_ADC2), U2.34 (GPIO28_ADC2); no longer U1.20 (GPIO15)
- net col8: now also U1.29 (GPIO22), U2.29 (GPIO22); no longer U1.24 (GPIO18)
- net data1RX: now also J1.R2
- net data1TX: now also J1.R1
- net encA: now also U2.22 (GPIO17)
- net encB: now also U2.21 (GPIO16)
- net row0: now also U2.4 (GPIO2)
- net row1: now also U2.5 (GPIO3)
- net row2: now also U2.6 (GPIO4)
- net row3: now also U2.7 (GPIO5)
- net row4: now also U2.9 (GPIO6)
- net row5: now also U2.10 (GPIO7)
- new net: D1.2 (A), U2.40 (VBUS)
- new net MI: J2.7 (Pin_7), U2.26 (GPIO20)
- new net MO: J2.6 (Pin_6), U2.25 (GPIO19)
- new net SC: J2.5 (Pin_5), U2.24 (GPIO18)
- new net SS: J2.4 (Pin_4), U2.27 (GPIO21)
- new net VI: J2.8 (Pin_8)
- new net data1RX_RH: J4.R1, U2.2 (GPIO1)
- new net data1TX_RH: J4.R2, U2.1 (GPIO0)
- no-connect marks 13 -> 20
Other:
- note added: "@todo - can the TX/RX Crossover be done in firmware, so serial fallback for TRS calbes is an option?"
- note added: "PMW3360 Trackball https://wylderbuilds.com/trackball-install"
- note removed: "Pimaroni Trackball"
- moved on the sheet: H1, H10, H11, H12, H13, H2, H3, H4, H5, H6, H7, H8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
