File: ergodonk_pico/ergodonk_pico.kicad_sch (KiCad schematic)
At the start: 338 parts, among them J1 AudioJack4, J2 Conn_01x08_Socket, J4 AudioJack4, Q1 TIP120, U1 Pico, U2 Pico

Commit message: Added 'simple' variant
Connections:
- net SW_LH_41_A: no longer U2.12 (GPIO9)
- net SW_RH_41_A: now also U2.12 (GPIO9)
- net col0: no longer U2.11 (GPIO8)
- net col0_rh: now also U2.11 (GPIO8)
- net col2: no longer U2.14 (GPIO10)
- net col2_rh: now also U2.14 (GPIO10)
- net col3: no longer U2.15 (GPIO11)
- net col3_rh: now also U2.15 (GPIO11)
- net col4: no longer U2.16 (GPIO12)
- net col4_rh: now also U2.16 (GPIO12)
- net col5: no longer U2.17 (GPIO13)
- net col5_rh: now also U2.17 (GPIO13)
- net col6: no longer U2.19 (GPIO14)
- net col6_rh: now also U2.19 (GPIO14)
- net col7: no longer U2.34 (GPIO28_ADC2)
- net col7_rh: now also U2.34 (GPIO28_ADC2)
- net col8: no longer U2.29 (GPIO22)
- net col8_rh: now also U2.29 (GPIO22)
- net encA: no longer SWRH_ROT1.A, U2.22 (GPIO17)
- net encB: no longer SWRH_ROT1.B, U2.21 (GPIO16)
- net row0: no longer U2.4 (GPIO2)
- net row0_rh: now also U2.4 (GPIO2)
- net row1: no longer U2.5 (GPIO3)
- net row1_rh: now also U2.5 (GPIO3)
- net row2: no longer U2.6 (GPIO4)
- net row2_rh: now also U2.6 (GPIO4)
- net row3: no longer U2.7 (GPIO5)
- net row3_rh: now also U2.7 (GPIO5)
- net row4: no longer U2.9 (GPIO6)
- net row4_rh: now also U2.9 (GPIO6)
- net row5: no longer U2.10 (GPIO7)
- net row5_rh: now also U2.10 (GPIO7)
- new net encA_rh: SWRH_ROT1.A, U2.22 (GPIO17)
- new net encB_rh: SWRH_ROT1.B, U2.21 (GPIO16)
Changed lines of the file:
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@@
     )
   )
-  (global_label "row0" (shape input) (at 306.07 -64.77 180)
+  (global_label "row0_rh" (shape input) (at 306.07 -64.77 180)
     (effects (font (size 1.27 1.27)) (justify right))
     (property "Intersheetrefs" "${INTERSHEET_REFS}" (at 306.07 -64.77 0)
@@
     )
   )
-  (global_label "col5" (shape input) (at 306.07 -31.75 180)
+  (global_label "col5_rh" (shape input) (at 306.07 -31.75 180)
     (effects (font (size 1.27 1.27)) (justify right))
     (property "Intersheetrefs" "${INTERSHEET_REFS}" (at 306.07 -31.75 0)
@@
     )
   )
-  (global_label "row2" (shape input) (at 306.07 -59.69 180)
+  (global_label "row2_rh" (shape input) (at 306.07 -59.69 180)
     (effects (font (size 1.27 1.27)) (justify right))
     (property "Intersheetrefs" "${INTERSHEET_REFS}" (at 306.07 -59.69 0)
@@
     )
   )
-  (global_label "col8" (shape input) (at 341.63 -44.45 0) (fields_autoplaced)
-    (effects (font (size 1.27 1.27)) (justify left))
-    (property "Intersheetrefs" "${INTERSHEET_REFS}" (at 348.6481 -44.45 0)
+  (global_label "col8_rh" (shape input) (at 341.63 -44.45 0) (fields_autoplaced)
+    (effects (font (size 1.27 1.27)) (justify left))
+    (property "Intersheetrefs" "${INTERSHEET_REFS}" (at 351.5509 -44.45 0)
       (effects (font (size 1.27 1.27)) (justify left) hide)
     )
@@
     )
   )
-  (global_label "row4" (shape input) (at 306.07 -52.07 180)
+  (global_label "row4_rh" (shape input) (at 306.07 -52.07 180)
     (effects (font (size 1.27 1.27)) (justify right))
     (property "Intersheetrefs" "${INTERSHEET_REFS}" (at 306.07 -52.07 0)
@@
     )
   )
-  (global_label "row5" (shape input) (at 306.07 -49.53 180) (fields_autoplaced)
-    (effects (font (size 1.27 1.27)) (justify right))
-    (property "Intersheetrefs" "${INTERSHEET_REFS}" (at 298.689 -49.53 0)
+  (global_label "row5_rh" (shape input) (at 306.07 -49.53 180) (fields_autoplaced)
+    (effects (font (size 1.27 1.27)) (justify right))
+    (property "Intersheetrefs" "${INTERSHEET_REFS}" (at 295.7862 -49.53 0)
       (effects (font (size 1.27 1.27)) (justify right) hide)
     )
@@
     )
   )
-  (global_label "col4" (shape input) (at 306.07 -34.29 180)
+  (global_label "col4_rh" (shape input) (at 306.07 -34.29 180)
     (effects (font (size 1.27 1.27)) (justify right))
     (property "Intersheetrefs" "${INTERSHEET_REFS}" (at 306.07 -34.29 0)
@@
     )
   )
-  (global_label "row1" (shape input) (at 306.07 -62.23 180)
+  (global_label "row1_rh" (shape input) (at 306.07 -62.23 180)
     (effects (font (size 1.27 1.27)) (justify right))
     (property "Intersheetrefs" "${INTERSHEET_REFS}" (at 306.07 -62.23 0)
@@
     )
   )
-  (global_label "col1" (shape input) (at 306.07 -44.45 180)
+  (global_label "col1_rh" (shape input) (at 306.07 -44.45 180)
     (effects (font (size 1.27 1.27)) (justify right))
     (property "Intersheetrefs" "${INTERSHEET_REFS}" (at 306.07 -44.45 0)
@@
     )
   )
-  (global_label "col3" (shape input) (at 306.07 -36.83 180)
+  (global_label "col3_rh" (shape input) (at 306.07 -36.83 180)
     (effects (font (size 1.27 1.27)) (justify right))
     (property "Intersheetrefs" "${INTERSHEET_REFS}" (at 306.07 -36.83 0)
@@
     )
   )
-  (global_label "encB" (shape input) (at 262.89 181.61 180) (fields_autoplaced)
-    (effects (font (size 1.27 1.27)) (justify right))
-    (property "Intersheetrefs" "${INTERSHEET_REFS}" (at 255.8807 181.5306 0)
+  (global_label "encB_rh" (shape input) (at 262.89 181.61 180) (fields_autoplaced)
+    (effects (font (size 1.27 1.27)) (justify right))
+    (property "Intersheetrefs" "${INTERSHEET_REFS}" (at 252.4852 181.61 0)
       (effects (font (size 1.27 1.27)) (justify right) hide)
     )
@@
     )
   )
-  (global_label "col7" (shape input) (at 341.63 -57.15 0) (fields_autoplaced)
-    (effects (font (size 1.27 1.27)) (justify left))
-    (property "Intersheetrefs" "${INTERSHEET_REFS}" (at 348.6481 -57.15 0)
+  (global_label "col7_rh" (shape input) (at 341.63 -57.15 0) (fields_autoplaced)
+    (effects (font (size 1.27 1.27)) (justify left))
+    (property "Intersheetrefs" "${INTERSHEET_REFS}" (at 351.5509 -57.15 0)
       (effects (font (size 1.27 1.27)) (justify left) hide)
     )
@@
     )
   )
-  (global_label "col6" (shape input) (at 306.07 -26.67 180) (fields_autoplaced)
-    (effects (font (size 1.27 1.27)) (justify right))
-    (property "Intersheetrefs" "${INTERSHEET_REFS}" (at 299.0519 -26.67 0)
+  (global_label "col6_rh" (shape input) (at 306.07 -26.67 180) (fields_autoplaced)
+    (effects (font (size 1.27 1.27)) (justify right))
+    (property "Intersheetrefs" "${INTERSHEET_REFS}" (at 296.1491 -26.67 0)
       (effects (font (size 1.27 1.27)) (justify right) hide)
     )
@@
     )
   )
-  (global_label "encA" (shape input) (at 341.63 -26.67 0)
+  (global_label "encA_rh" (shape input) (at 341.63 -26.67 0)
     (effects (font (size 1.27 1.27)) (justify left))
     (property "Intersheetrefs" "${INTERSHEET_REFS}" (at 341.63 -26.67 0)
@@
     )
   )
-  (global_label "row3" (shape input) (at 306.07 -57.15 180)
+  (global_label "row3_rh" (shape input) (at 306.07 -57.15 180)
     (effects (font (size 1.27 1.27)) (justify right))
     (property "Intersheetrefs" "${INTERSHEET_REFS}" (at 306.07 -57.15 0)
@@
     )
   )
-  (global_label "col2" (shape input) (at 306.07 -39.37 180)
+  (global_label "col2_rh" (shape input) (at 306.07 -39.37 180)
     (effects (font (size 1.27 1.27)) (justify right))
     (property "Intersheetrefs" "${INTERSHEET_REFS}" (at 306.07 -39.37 0)
@@
     )
   )
-  (global_label "encB" (shape input) (at 341.63 -24.13 0)
+  (global_label "encB_rh" (shape input) (at 341.63 -24.13 0)
     (effects (font (size 1.27 1.27)) (justify left))
     (property "Intersheetrefs" "${INTERSHEET_REFS}" (at 341.63 -24.13 0)
@@
     )
   )
-  (global_label "col0" (shape input) (at 306.07 -46.99 180)
+  (global_label "col0_rh" (shape input) (at 306.07 -46.99 180)
     (effects (font (size 1.27 1.27)) (justify right))
     (property "Intersheetrefs" "${INTERSHEET_REFS}" (at 306.07 -46.99 0)
@@
     )
   )
-  (global_label "encA" (shape input) (at 259.08 176.53 180) (fields_autoplaced)
-    (effects (font (size 1.27 1.27)) (justify right))
-    (property "Intersheetrefs" "${INTERSHEET_REFS}" (at 252.2521 176.4506 0)
-      (effects (font (size 1.27 1.27)) (justify right) hide)
-    )
+  (global_label "encA_rh" (shape input) (at 259.08 176.53 180) (fields_autoplaced)
+    (effects (font (size 1.27 1.27)) (justify right))
+    (property "Intersheetrefs" "${INTERSHEET_REFS}" (at 248.8566 176.53 0)
+      (effects (font (size 1.27 1.27)) (justify right) hide)
+    )
