File: ergodonk_pico/ergodonk_pico.kicad_pcb (KiCad board)
At the start: 2 copper layers, 216.5 x 156.6 mm, 467 parts, among them J10 Pimaroni Trackball, J11 4PIN, J2 Pimaroni Trackball, J3 AudioJack4, Q1 TIP120, SW08_RH10 SW_PUSH_LED, SW1 SW_PUSH_LED, SW10 SW_PUSH_LED, SW11 SW_PUSH_LED, SW12 SW_PUSH_LED, SW13 SW_PUSH_LED, SW14 SW_PUSH_LED, SW15 SW_PUSH_LED, SW16 SW_PUSH_LED, SW17 SW_PUSH_LED, SW18_RH10 SW_PUSH_LED, SW2 SW_PUSH_LED, SW20 SW_PUSH_LED, SW21 SW_PUSH_LED, SW22 SW_PUSH_LED, SW23 SW_PUSH_LED, SW24 SW_PUSH_LED, SW25 SW_PUSH_LED, SW26 SW_PUSH_LED, SW27 SW_PUSH_LED, SW28_RH10 SW_PUSH_LED, SW3 SW_PUSH_LED, SW30 SW_PUSH_LED, SW31 SW_PUSH_LED, SW32 SW_PUSH_LED, SW33 SW_PUSH_LED, SW34 SW_PUSH_LED, SW35 SW_PUSH_LED, SW36 SW_PUSH_LED, SW37 SW_PUSH_LED, SW38_RH10 SW_PUSH_LED, SW4 SW_PUSH_LED, SW40 SW_PUSH_LED, SW42 SW_PUSH_LED, SW43 SW_PUSH_LED, SW44 SW_PUSH_LED, SW45 SW_PUSH_LED, SW46 SW_PUSH_LED, SW47 SW_PUSH_LED, SW48_RH10 SW_PUSH_LED, SW5 SW_PUSH_LED, SW50 SW_PUSH_LED, SW51 SW_PUSH_LED, SW52 SW_PUSH_LED, SW53 SW_PUSH_LED, SW54 SW_PUSH_LED, SW55 SW_PUSH_LED, SW56 SW_PUSH_LED, SW57 SW_PUSH_LED, SW58 SW_PUSH_LED, SW6 SW_PUSH_LED, SW7 SW_PUSH_LED, U2 Pico

Commit message: Thumb rotation diode placement added tenting puck symbols and footprint
Parts:
- removed ?: , clipboard:7f3053b2-006a-4efc-aa06-df19745f0381
- removed D08_RH10, D1, D10, D11, D12, D13, D14, D15, D16, D17, D18_RH10, D2, D20, D21, D22, D23, D24, D25, D26, D27, D28_RH10, D3, D30, D31, D32, D33, D34, D35, D36, D37, D38_RH10, D4, D40, D41, D42, D43, D44, D45, D46, D47, D48_RH10, D5, D50, D51, D52, D53, D54, D55, D56, D57, D58, D6, D7: D, ergodonk_kicad_library:D_SOD-123_DO-35_Hybrid_DoubleSided
- removed the D_SOL_1 at (-514.4, -153.1)
- removed the H1 at (-469.1, -162.1)
- removed the H10 at (-470.9, -128.9)
- removed the H11 at (-412.5, -123.3)
- removed the H12 at (-545.6, -68.3)
- removed the H13 at (-566.8, -137.6)
- removed the H3 at (-356.5, -92.8)
- removed the H4 at (-397.1, -39.4)
- removed the H5 at (-431.0, -73.3)
- removed the H6 at (-458.0, -55.0)
- removed the H7 at (-521.5, -66.4)
- removed the H8 at (-509.9, -113.5)
- removed the H9 at (-529.8, -174.0)
- removed J10: Pimaroni Trackball, ergodonk_kicad_library:pimoroni_trackball
- removed J11: 4PIN, ergodonk_kicad_library:MJ-4PP-9_CANTOR_KITCHEN_SINK
- removed JP3: LH LED's, Connector_PinHeader_2.54mm:PinHeader_1x02_P2.54mm_Vertical
- removed the J_SOL_1 at (-503.7, -150.8)
- removed LS10: AST1109MLTRQ_MAL, ergodonk_kicad_library:AST1109MLTRQ
- removed OL10: OLED, ergodonk_kicad_library:OLED SSD1306 128x64 UNVERIFIED
- removed the Q1 at (-534.3, -156.4)
- removed R2: 1k, Resistor_THT:R_Axial_DIN0309_L9.0mm_D3.2mm_P12.70mm_Horizontal
- removed REF** (x3): RPi_Pico_SMD_TH - Junco, ergodonk_kicad_library:RPi_Pico_SMD_TH - Junco
- removed REF**: Tenting Puck, ergodonk_kicad_library:Tenting_Puck.kicad_mod_nocenter
- removed the S1 at (-489.9, -159.7)
- removed SW08_RH10: SW_PUSH_LED, ergodonk_kicad_library:V2_CherryMX_DoubleSided_Hotswap_miniE_2u_RH_ONLY
- removed SW1, SW10, SW11, SW12, SW13, SW14, SW15, SW16, SW17, SW2 (x2), SW20, SW21, SW22, SW23, SW24, SW25, SW26, SW3, SW30, SW31, SW32, SW33, SW34, SW35, SW36, SW4, SW40, SW42, SW43, SW44, SW45, SW46, SW5, SW50, SW54, SW55, SW56, SW6, SW7: SW_PUSH_LED, ergodonk_kicad_library:V2_CherryMX_DoubleSided_Hotswap_miniE
- removed SW18_RH10, SW38_RH10: SW_PUSH_LED, ergodonk_kicad_library:V2_CherryMX_DS_Hotswap_miniE_1U_SEED_RH
- removed SW27: SW_PUSH_LED, ergodonk_kicad_library:V2_CherryMX_DoubleSided_Hotswap_miniE_1.5u_LH_1u_RH
- removed SW28_RH10: SW_PUSH_LED, ergodonk_kicad_library:V2_CherryMX_DoubleSided_Hotswap_miniE_1.5u_RH_ONLY
- removed SW37: SW_PUSH_LED, ergodonk_kicad_library:V2_CherryMX_DoubleSided_Hotswap_miniE_1.75u_LH_1u_RH
- removed SW47: SW_PUSH_LED, ergodonk_kicad_library:V2_CherryMX_DoubleSided_Hotswap_miniE_2.25u_LH_2.75u_RH
- removed SW48_RH10: SW_PUSH_LED, ergodonk_kicad_library:V2_CherryMX_DoubleSided_Hotswap_miniE_2.25u_RH_ONLY
- removed SW51, SW52: SW_PUSH_LED, ergodonk_kicad_library:V2_CherryMX_DoubleSided_Hotswap_miniE_2u_Vertical
- removed SW53: SW_PUSH_LED, ergodonk_kicad_library:V2_CherryMX_DoubleSided_Hotswap_miniE_1.25u_Vertical
- removed SW57, SW58: SW_PUSH_LED, ergodonk_kicad_library:V2_CherryMX_DoubleSided_Hotswap_miniE_1.25u
- removed the SWLH_ROT1 at (-392.9, -85.4)
- added H14: Tenting puck mount, ergodonk_kicad_library:Tenting_Puck.kicad_mod_nocenter, F.Cu at (-51.6, 58.1)
- added H15: Tenting puck mount, ergodonk_kicad_library:Tenting_Puck.kicad_mod_nocenter, F.Cu at (-51.6, 101.6)
- L_LH_00, L_LH_1, L_LH_10, L_LH_11, L_LH_12, L_LH_13, L_LH_14, L_LH_15, L_LH_16, L_LH_17, L_LH_2, L_LH_20, L_LH_21, L_LH_22, L_LH_23, L_LH_24, L_LH_25, L_LH_26, L_LH_27, L_LH_3, L_LH_30, L_LH_31, L_LH_32, L_LH_33, L_LH_34, L_LH_35, L_LH_36, L_LH_37, L_LH_4, L_LH_40, L_LH_41, L_LH_42, L_LH_43, L_LH_44, L_LH_45, L_LH_46, L_LH_47, L_LH_5, L_LH_50, L_LH_51, L_LH_52, L_LH_53, L_LH_54, L_LH_55, L_LH_56, L_LH_57, L_LH_58, L_LH_6, L_LH_7, L_RH_00, L_RH_1, L_RH_10, L_RH_11, L_RH_12, L_RH_13, L_RH_14, L_RH_15, L_RH_16, L_RH_17, L_RH_18, L_RH_2, L_RH_20, L_RH_21, L_RH_22, L_RH_23, L_RH_24, L_RH_25, L_RH_26, L_RH_27, L_RH_28, L_RH_3, L_RH_30, L_RH_31, L_RH_32, L_RH_33, L_RH_34, L_RH_35, L_RH_36, L_RH_37, L_RH_38, L_RH_4, L_RH_40, L_RH_41, L_RH_42, L_RH_43, L_RH_44, L_RH_45, L_RH_46, L_RH_47, L_RH_48, L_RH_5, L_RH_50, L_RH_51, L_RH_52, L_RH_53, L_RH_54, L_RH_55, L_RH_56, L_RH_57, L_RH_58, L_RH_6, L_RH_7, L_RH_8: footprint ergodonk_pico:V2_CherryMX_Hotswap -> ergodonk_pico:SK6812-MINI-E
- SW_RH_32: footprint ergodonk_pico:Chunky_2040_footprint_ergodonk_customs -> ergodonk_pico:V2_CherryMX_Hotswap
- SW_RH_51, SW_RH_52: footprint ergodonk_pico:V2_CherryMX_Hotswap -> ergodonk_pico:V2_CherryMX_KailhV2_Hotswap
- moved D_RH_14 507.3 mm to (73.0, -92.4)
- moved D_RH_48 506.6 mm to (161.1, -39.3)
- moved D_RH_37 499.6 mm to (130.2, -39.3)
- moved D_LH_02 494.0 mm to (-14.9, -163.4)
- moved D_LH_03 494.0 mm to (-14.9, -161.1)
- moved D_LH_04 494.0 mm to (-14.9, -158.8)
- moved D_LH_07 494.0 mm to (-14.9, -151.9)
- moved D_LH_10 494.0 mm to (-14.9, -149.6)
- moved D_LH_11 494.0 mm to (-14.9, -147.3)
- moved D_LH_14 494.0 mm to (-14.9, -140.4)
- moved D_LH_15 494.0 mm to (-14.9, -138.1)
- moved D_LH_16 494.0 mm to (-14.9, -135.8)
- moved D_LH_21 494.0 mm to (-14.9, -128.9)
- moved D_LH_22 494.0 mm to (-14.9, -126.6)
- moved D_LH_23 494.0 mm to (-14.9, -124.3)
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Connections:
- D_RH_32 pad 2: unconnected-(D_RH_32-A-Pad2) -> Net-(D_RH_32-A)
- L_LH_00 pad 1: (no net) -> VDD
- L_LH_00 pad 2: (no net) -> unconnected-(L_LH_00-DOUT-Pad2)
- L_LH_1 pad 1: (no net) -> VDD
- L_LH_1 pad 2: (no net) -> unconnected-(L_LH_1-DOUT-Pad2)
- L_LH_10 pad 1: (no net) -> VDD
- L_LH_10 pad 2: (no net) -> unconnected-(L_LH_10-DOUT-Pad2)
- L_LH_11 pad 1: (no net) -> VDD
- L_LH_11 pad 2: (no net) -> unconnected-(L_LH_11-DOUT-Pad2)
- L_LH_12 pad 1: (no net) -> VDD
- L_LH_12 pad 2: (no net) -> unconnected-(L_LH_12-DOUT-Pad2)
- L_LH_13 pad 1: (no net) -> VDD
- L_LH_13 pad 2: (no net) -> unconnected-(L_LH_13-DOUT-Pad2)
- L_LH_14 pad 1: (no net) -> VDD
- L_LH_14 pad 2: (no net) -> unconnected-(L_LH_14-DOUT-Pad2)
- L_LH_15 pad 1: (no net) -> VDD
- L_LH_15 pad 2: (no net) -> unconnected-(L_LH_15-DOUT-Pad2)
- L_LH_16 pad 1: (no net) -> VDD
- L_LH_16 pad 2: (no net) -> unconnected-(L_LH_16-DOUT-Pad2)
- L_LH_17 pad 1: (no net) -> VDD
- L_LH_17 pad 2: (no net) -> unconnected-(L_LH_17-DOUT-Pad2)
- L_LH_2 pad 1: (no net) -> VDD
- L_LH_2 pad 2: (no net) -> unconnected-(L_LH_2-DOUT-Pad2)
- L_LH_20 pad 1: (no net) -> VDD
- L_LH_20 pad 2: (no net) -> unconnected-(L_LH_20-DOUT-Pad2)
- L_LH_21 pad 1: (no net) -> VDD
- L_LH_21 pad 2: (no net) -> unconnected-(L_LH_21-DOUT-Pad2)
- L_LH_22 pad 1: (no net) -> VDD
- L_LH_22 pad 2: (no net) -> unconnected-(L_LH_22-DOUT-Pad2)
- L_LH_23 pad 1: (no net) -> VDD
- L_LH_23 pad 2: (no net) -> unconnected-(L_LH_23-DOUT-Pad2)
- L_LH_24 pad 1: (no net) -> VDD
- L_LH_24 pad 2: (no net) -> unconnected-(L_LH_24-DOUT-Pad2)
- L_LH_25 pad 1: (no net) -> VDD
- L_LH_25 pad 2: (no net) -> unconnected-(L_LH_25-DOUT-Pad2)
- L_LH_26 pad 1: (no net) -> VDD
- L_LH_26 pad 2: (no net) -> unconnected-(L_LH_26-DOUT-Pad2)
- L_LH_27 pad 1: (no net) -> VDD
- L_LH_27 pad 2: (no net) -> unconnected-(L_LH_27-DOUT-Pad2)
- L_LH_3 pad 1: (no net) -> VDD
- L_LH_3 pad 2: (no net) -> unconnected-(L_LH_3-DOUT-Pad2)
- L_LH_30 pad 1: (no net) -> VDD
- L_LH_30 pad 2: (no net) -> unconnected-(L_LH_30-DOUT-Pad2)
- L_LH_31 pad 1: (no net) -> VDD
- L_LH_31 pad 2: (no net) -> unconnected-(L_LH_31-DOUT-Pad2)
- L_LH_32 pad 1: (no net) -> VDD
- L_LH_32 pad 2: (no net) -> unconnected-(L_LH_32-DOUT-Pad2)
- L_LH_33 pad 1: (no net) -> VDD
- L_LH_33 pad 2: (no net) -> unconnected-(L_LH_33-DOUT-Pad2)
- L_LH_34 pad 1: (no net) -> VDD
- L_LH_34 pad 2: (no net) -> unconnected-(L_LH_34-DOUT-Pad2)
- L_LH_35 pad 1: (no net) -> VDD
- L_LH_35 pad 2: (no net) -> unconnected-(L_LH_35-DOUT-Pad2)
- L_LH_36 pad 1: (no net) -> VDD
- L_LH_36 pad 2: (no net) -> unconnected-(L_LH_36-DOUT-Pad2)
- L_LH_37 pad 1: (no net) -> VDD
- L_LH_37 pad 2: (no net) -> unconnected-(L_LH_37-DOUT-Pad2)
- L_LH_4 pad 1: (no net) -> VDD
- L_LH_4 pad 2: (no net) -> unconnected-(L_LH_4-DOUT-Pad2)
- L_LH_40 pad 1: (no net) -> VDD
- L_LH_40 pad 2: (no net) -> unconnected-(L_LH_40-DOUT-Pad2)
- L_LH_41 pad 1: (no net) -> VDD
- L_LH_41 pad 2: (no net) -> unconnected-(L_LH_41-DOUT-Pad2)
- L_LH_42 pad 1: (no net) -> VDD
- L_LH_42 pad 2: (no net) -> unconnected-(L_LH_42-DOUT-Pad2)
- L_LH_43 pad 1: (no net) -> VDD
- L_LH_43 pad 2: (no net) -> unconnected-(L_LH_43-DOUT-Pad2)
- L_LH_44 pad 1: (no net) -> VDD
- L_LH_44 pad 2: (no net) -> unconnected-(L_LH_44-DOUT-Pad2)
- L_LH_45 pad 1: (no net) -> VDD
- L_LH_45 pad 2: (no net) -> unconnected-(L_LH_45-DOUT-Pad2)
- L_LH_46 pad 1: (no net) -> VDD
- L_LH_46 pad 2: (no net) -> unconnected-(L_LH_46-DOUT-Pad2)
- L_LH_47 pad 1: (no net) -> VDD
- L_LH_47 pad 2: (no net) -> unconnected-(L_LH_47-DOUT-Pad2)
- L_LH_5 pad 1: (no net) -> VDD
- L_LH_5 pad 2: (no net) -> unconnected-(L_LH_5-DOUT-Pad2)
- L_LH_50 pad 1: (no net) -> VDD
- L_LH_50 pad 2: (no net) -> unconnected-(L_LH_50-DOUT-Pad2)
- L_LH_51 pad 1: (no net) -> VDD
- L_LH_51 pad 2: (no net) -> unconnected-(L_LH_51-DOUT-Pad2)
- L_LH_52 pad 1: (no net) -> VDD
- L_LH_52 pad 2: (no net) -> unconnected-(L_LH_52-DOUT-Pad2)
- L_LH_53 pad 1: (no net) -> VDD
- L_LH_53 pad 2: (no net) -> unconnected-(L_LH_53-DOUT-Pad2)
- L_LH_54 pad 1: (no net) -> VDD
- L_LH_54 pad 2: (no net) -> unconnected-(L_LH_54-DOUT-Pad2)
- L_LH_55 pad 1: (no net) -> VDD
- L_LH_55 pad 2: (no net) -> unconnected-(L_LH_55-DOUT-Pad2)
- L_LH_56 pad 1: (no net) -> VDD
- L_LH_56 pad 2: (no net) -> unconnected-(L_LH_56-DOUT-Pad2)
- L_LH_57 pad 1: (no net) -> VDD
- L_LH_57 pad 2: (no net) -> unconnected-(L_LH_57-DOUT-Pad2)
- L_LH_58 pad 1: (no net) -> VDD
- L_LH_58 pad 2: (no net) -> unconnected-(L_LH_58-DOUT-Pad2)
- L_LH_6 pad 1: (no net) -> VDD
- L_LH_6 pad 2: (no net) -> unconnected-(L_LH_6-DOUT-Pad2)
- L_LH_7 pad 1: (no net) -> VDD
- L_LH_7 pad 2: (no net) -> unconnected-(L_LH_7-DOUT-Pad2)
- L_RH_00 pad 1: (no net) -> VDD
- L_RH_00 pad 2: (no net) -> unconnected-(L_RH_00-DOUT-Pad2)
- L_RH_1 pad 1: (no net) -> VDD
- L_RH_1 pad 2: (no net) -> unconnected-(L_RH_1-DOUT-Pad2)
- L_RH_10 pad 1: (no net) -> VDD
- L_RH_10 pad 2: (no net) -> unconnected-(L_RH_10-DOUT-Pad2)
- L_RH_11 pad 1: (no net) -> VDD
- L_RH_11 pad 2: (no net) -> unconnected-(L_RH_11-DOUT-Pad2)
- L_RH_12 pad 1: (no net) -> VDD
- L_RH_12 pad 2: (no net) -> unconnected-(L_RH_12-DOUT-Pad2)
- L_RH_13 pad 1: (no net) -> VDD
- L_RH_13 pad 2: (no net) -> unconnected-(L_RH_13-DOUT-Pad2)
- L_RH_14 pad 1: (no net) -> VDD
- L_RH_14 pad 2: (no net) -> unconnected-(L_RH_14-DOUT-Pad2)
- L_RH_15 pad 1: (no net) -> VDD
- L_RH_15 pad 2: (no net) -> unconnected-(L_RH_15-DOUT-Pad2)
- L_RH_16 pad 1: (no net) -> VDD
- L_RH_16 pad 2: (no net) -> unconnected-(L_RH_16-DOUT-Pad2)
- L_RH_17 pad 1: (no net) -> VDD
- L_RH_17 pad 2: (no net) -> unconnected-(L_RH_17-DOUT-Pad2)
- L_RH_18 pad 1: (no net) -> VDD
- L_RH_18 pad 2: (no net) -> unconnected-(L_RH_18-DOUT-Pad2)
- L_RH_2 pad 1: (no net) -> VDD
- L_RH_2 pad 2: (no net) -> unconnected-(L_RH_2-DOUT-Pad2)
- L_RH_20 pad 1: (no net) -> VDD
- L_RH_20 pad 2: (no net) -> unconnected-(L_RH_20-DOUT-Pad2)
- L_RH_21 pad 1: (no net) -> VDD
- L_RH_21 pad 2: (no net) -> unconnected-(L_RH_21-DOUT-Pad2)
- L_RH_22 pad 1: (no net) -> VDD
- L_RH_22 pad 2: (no net) -> unconnected-(L_RH_22-DOUT-Pad2)
- L_RH_23 pad 1: (no net) -> VDD
- L_RH_23 pad 2: (no net) -> unconnected-(L_RH_23-DOUT-Pad2)
- L_RH_24 pad 1: (no net) -> VDD
- L_RH_24 pad 2: (no net) -> unconnected-(L_RH_24-DOUT-Pad2)
- L_RH_25 pad 1: (no net) -> VDD
- L_RH_25 pad 2: (no net) -> unconnected-(L_RH_25-DOUT-Pad2)
- L_RH_26 pad 1: (no net) -> VDD
- L_RH_26 pad 2: (no net) -> unconnected-(L_RH_26-DOUT-Pad2)
- L_RH_27 pad 1: (no net) -> VDD
- L_RH_27 pad 2: (no net) -> unconnected-(L_RH_27-DOUT-Pad2)
- L_RH_28 pad 1: (no net) -> VDD
- L_RH_28 pad 2: (no net) -> unconnected-(L_RH_28-DOUT-Pad2)
- L_RH_3 pad 1: (no net) -> VDD
- L_RH_3 pad 2: (no net) -> unconnected-(L_RH_3-DOUT-Pad2)
- L_RH_30 pad 1: (no net) -> VDD
- L_RH_30 pad 2: (no net) -> unconnected-(L_RH_30-DOUT-Pad2)
- L_RH_31 pad 1: (no net) -> VDD
- L_RH_31 pad 2: (no net) -> unconnected-(L_RH_31-DOUT-Pad2)
- L_RH_32 pad 1: (no net) -> VDD
- L_RH_32 pad 2: (no net) -> unconnected-(L_RH_32-DOUT-Pad2)
- L_RH_33 pad 1: (no net) -> VDD
- L_RH_33 pad 2: (no net) -> unconnected-(L_RH_33-DOUT-Pad2)
- L_RH_34 pad 1: (no net) -> VDD
- L_RH_34 pad 2: (no net) -> unconnected-(L_RH_34-DOUT-Pad2)
- L_RH_35 pad 1: (no net) -> VDD
- L_RH_35 pad 2: (no net) -> unconnected-(L_RH_35-DOUT-Pad2)
- L_RH_36 pad 1: (no net) -> VDD
- L_RH_36 pad 2: (no net) -> unconnected-(L_RH_36-DOUT-Pad2)
- L_RH_37 pad 1: (no net) -> VDD
- L_RH_37 pad 2: (no net) -> unconnected-(L_RH_37-DOUT-Pad2)
- L_RH_38 pad 1: (no net) -> VDD
- L_RH_38 pad 2: (no net) -> unconnected-(L_RH_38-DOUT-Pad2)
- L_RH_4 pad 1: (no net) -> VDD
- L_RH_4 pad 2: (no net) -> unconnected-(L_RH_4-DOUT-Pad2)
- L_RH_40 pad 1: (no net) -> VDD
- L_RH_40 pad 2: (no net) -> unconnected-(L_RH_40-DOUT-Pad2)
- L_RH_41 pad 1: (no net) -> VDD
- L_RH_41 pad 2: (no net) -> unconnected-(L_RH_41-DOUT-Pad2)
- L_RH_42 pad 1: (no net) -> VDD
- L_RH_42 pad 2: (no net) -> unconnected-(L_RH_42-DOUT-Pad2)
- L_RH_43 pad 1: (no net) -> VDD
- L_RH_43 pad 2: (no net) -> unconnected-(L_RH_43-DOUT-Pad2)
- L_RH_44 pad 1: (no net) -> VDD
- L_RH_44 pad 2: (no net) -> unconnected-(L_RH_44-DOUT-Pad2)
- L_RH_45 pad 1: (no net) -> VDD
- L_RH_45 pad 2: (no net) -> unconnected-(L_RH_45-DOUT-Pad2)
- L_RH_46 pad 1: (no net) -> VDD
- L_RH_46 pad 2: (no net) -> unconnected-(L_RH_46-DOUT-Pad2)
- L_RH_47 pad 1: (no net) -> VDD
- L_RH_47 pad 2: (no net) -> unconnected-(L_RH_47-DOUT-Pad2)
- L_RH_48 pad 1: (no net) -> VDD
- L_RH_48 pad 2: (no net) -> unconnected-(L_RH_48-DOUT-Pad2)
- L_RH_5 pad 1: (no net) -> VDD
- L_RH_5 pad 2: (no net) -> unconnected-(L_RH_5-DOUT-Pad2)
- L_RH_50 pad 1: (no net) -> VDD
- L_RH_50 pad 2: (no net) -> unconnected-(L_RH_50-DOUT-Pad2)
- L_RH_51 pad 1: (no net) -> VDD
- L_RH_51 pad 2: (no net) -> unconnected-(L_RH_51-DOUT-Pad2)
- L_RH_52 pad 1: (no net) -> VDD
- L_RH_52 pad 2: (no net) -> unconnected-(L_RH_52-DOUT-Pad2)
- L_RH_53 pad 1: (no net) -> VDD
- L_RH_53 pad 2: (no net) -> unconnected-(L_RH_53-DOUT-Pad2)
- L_RH_54 pad 1: (no net) -> VDD
- L_RH_54 pad 2: (no net) -> unconnected-(L_RH_54-DOUT-Pad2)
- L_RH_55 pad 1: (no net) -> VDD
- L_RH_55 pad 2: (no net) -> unconnected-(L_RH_55-DOUT-Pad2)
- L_RH_56 pad 1: (no net) -> VDD
- L_RH_56 pad 2: (no net) -> unconnected-(L_RH_56-DOUT-Pad2)
- L_RH_57 pad 1: (no net) -> VDD
- L_RH_57 pad 2: (no net) -> unconnected-(L_RH_57-DOUT-Pad2)
- L_RH_58 pad 1: (no net) -> VDD
- L_RH_58 pad 2: (no net) -> unconnected-(L_RH_58-DOUT-Pad2)
- L_RH_6 pad 1: (no net) -> VDD
- L_RH_6 pad 2: (no net) -> unconnected-(L_RH_6-DOUT-Pad2)
- L_RH_7 pad 1: (no net) -> VDD
- L_RH_7 pad 2: (no net) -> unconnected-(L_RH_7-DOUT-Pad2)
- L_RH_8 pad 1: (no net) -> VDD
- L_RH_8 pad 2: (no net) -> unconnected-(L_RH_8-DOUT-Pad2)
- SW_LH_00 pad 1: (no net) -> col0
- SW_LH_00 pad 2: (no net) -> Net-(D_LH_00-A)
- SW_LH_01 pad 1: (no net) -> SW_LH_41_A
- SW_LH_01 pad 2: (no net) -> Net-(D_LH_01-A)
- SW_LH_02 pad 1: (no net) -> col2
- SW_LH_02 pad 2: (no net) -> Net-(D_LH_02-A)
- SW_LH_03 pad 1: (no net) -> col3
- SW_LH_03 pad 2: (no net) -> Net-(D_LH_03-A)
- SW_LH_04 pad 1: (no net) -> col4
- SW_LH_04 pad 2: (no net) -> Net-(D_LH_04-A)
- SW_LH_05 pad 1: (no net) -> col5
- SW_LH_05 pad 2: (no net) -> Net-(D_LH_05-A)
- SW_LH_06 pad 1: (no net) -> col6
- SW_LH_06 pad 2: (no net) -> Net-(D_LH_06-A)
- SW_LH_07 pad 1: (no net) -> col7
- SW_LH_07 pad 2: (no net) -> Net-(D_LH_07-A)
- SW_LH_10 pad 1: (no net) -> col0
- SW_LH_10 pad 2: (no net) -> Net-(D_LH_10-A)
- SW_LH_11 pad 1: (no net) -> SW_LH_41_A
- SW_LH_11 pad 2: (no net) -> Net-(D_LH_11-A)
- SW_LH_12 pad 1: (no net) -> col2
- SW_LH_12 pad 2: (no net) -> Net-(D_LH_12-A)
- SW_LH_13 pad 1: (no net) -> col3
- SW_LH_13 pad 2: (no net) -> Net-(D_LH_13-A)
- SW_LH_14 pad 1: (no net) -> col4
- SW_LH_14 pad 2: (no net) -> Net-(D_LH_14-A)
- SW_LH_15 pad 1: (no net) -> col5
- SW_LH_15 pad 2: (no net) -> Net-(D_LH_15-A)
- SW_LH_16 pad 1: (no net) -> col6
- SW_LH_16 pad 2: (no net) -> Net-(D_LH_16-A)
- SW_LH_17 pad 1: (no net) -> col7
- SW_LH_17 pad 2: (no net) -> Net-(D_LH_17-A)
- SW_LH_20 pad 1: (no net) -> col0
- SW_LH_20 pad 2: (no net) -> Net-(D_LH_20-A)
- SW_LH_21 pad 1: (no net) -> SW_LH_41_A
- SW_LH_21 pad 2: (no net) -> Net-(D_LH_21-A)
- SW_LH_22 pad 1: (no net) -> col2
- SW_LH_22 pad 2: (no net) -> Net-(D_LH_22-A)
- SW_LH_23 pad 1: (no net) -> col3
- SW_LH_23 pad 2: (no net) -> Net-(D_LH_23-A)
- SW_LH_24 pad 1: (no net) -> col4
- SW_LH_24 pad 2: (no net) -> Net-(D_LH_24-A)
- SW_LH_25 pad 1: (no net) -> col5
- SW_LH_25 pad 2: (no net) -> Net-(D_LH_25-A)
- SW_LH_26 pad 1: (no net) -> col6
- SW_LH_26 pad 2: (no net) -> Net-(D_LH_26-A)
- SW_LH_27 pad 1: (no net) -> col7
- SW_LH_27 pad 2: (no net) -> Net-(D_LH_27-A)
- SW_LH_30 pad 1: (no net) -> col0
- SW_LH_30 pad 2: (no net) -> Net-(D_LH_30-A)
- SW_LH_31 pad 1: (no net) -> SW_LH_41_A
- SW_LH_31 pad 2: (no net) -> Net-(D_LH_31-A)
- SW_LH_32 pad 1: (no net) -> col2
- SW_LH_32 pad 2: (no net) -> Net-(D_LH_32-A)
- SW_LH_33 pad 1: (no net) -> col3
- SW_LH_33 pad 2: (no net) -> Net-(D_LH_33-A)
- SW_LH_34 pad 1: (no net) -> col4
- SW_LH_34 pad 2: (no net) -> Net-(D_LH_34-A)
- SW_LH_35 pad 1: (no net) -> col5
- SW_LH_35 pad 2: (no net) -> Net-(D_LH_35-A)
- SW_LH_36 pad 1: (no net) -> col6
- SW_LH_36 pad 2: (no net) -> Net-(D_LH_36-A)
- SW_LH_37 pad 1: (no net) -> col7
- SW_LH_37 pad 2: (no net) -> Net-(D_LH_37-A)
- SW_LH_40 pad 1: (no net) -> col0
- SW_LH_40 pad 2: (no net) -> Net-(D_LH_40-A)
- SW_LH_42 pad 1: (no net) -> col2
- SW_LH_42 pad 2: (no net) -> Net-(D_LH_42-A)
- SW_LH_43 pad 1: (no net) -> col3
- SW_LH_43 pad 2: (no net) -> Net-(D_LH_43-A)
- SW_LH_44 pad 1: (no net) -> col4
- SW_LH_44 pad 2: (no net) -> Net-(D_LH_44-A)
- SW_LH_45 pad 1: (no net) -> col5
- SW_LH_45 pad 2: (no net) -> Net-(D_LH_45-A)
- SW_LH_46 pad 1: (no net) -> col6
- SW_LH_46 pad 2: (no net) -> Net-(D_LH_46-A)
- SW_LH_47 pad 1: (no net) -> col7
- SW_LH_47 pad 2: (no net) -> Net-(D_LH_47-A)
- SW_LH_50 pad 1: (no net) -> col0
- SW_LH_50 pad 2: (no net) -> Net-(D_LH_50-A)
- SW_LH_51 pad 1: (no net) -> SW_LH_41_A
- SW_LH_51 pad 2: (no net) -> Net-(D_LH_51-A)
- SW_LH_52 pad 1: (no net) -> col2
- SW_LH_52 pad 2: (no net) -> Net-(D_LH_52-A)
- SW_LH_53 pad 1: (no net) -> col3
- SW_LH_53 pad 2: (no net) -> Net-(D_LH_53-A)
- SW_LH_54 pad 1: (no net) -> col4
- SW_LH_54 pad 2: (no net) -> Net-(D_LH_54-A)
- SW_LH_55 pad 1: (no net) -> col5
- SW_LH_55 pad 2: (no net) -> Net-(D_LH_55-A)
- SW_LH_56 pad 1: (no net) -> col6
- SW_LH_56 pad 2: (no net) -> Net-(D_LH_56-A)
- SW_LH_57 pad 1: (no net) -> col7
- SW_LH_57 pad 2: (no net) -> Net-(D_LH_57-A)
- SW_LH_58 pad 1: (no net) -> col8
- SW_LH_58 pad 2: (no net) -> Net-(D_LH_58-A)
- SW_RH_00 pad 1: (no net) -> col0_rh
- SW_RH_00 pad 2: (no net) -> Net-(D_RH_00-A)
- SW_RH_01 pad 1: (no net) -> SW_RH_41_A
- SW_RH_01 pad 2: (no net) -> Net-(D_RH_01-A)
- SW_RH_02 pad 1: (no net) -> col2_rh
- SW_RH_02 pad 2: (no net) -> Net-(D_RH_02-A)
- SW_RH_03 pad 1: (no net) -> col3_rh
- SW_RH_03 pad 2: (no net) -> Net-(D_RH_03-A)
- SW_RH_04 pad 1: (no net) -> col4_rh
- SW_RH_04 pad 2: (no net) -> Net-(D_RH_04-A)
- SW_RH_05 pad 1: (no net) -> col5_rh
- SW_RH_05 pad 2: (no net) -> Net-(D_RH_05-A)
- SW_RH_06 pad 1: (no net) -> col6_rh
- SW_RH_06 pad 2: (no net) -> Net-(D_RH_06-A)
- SW_RH_07 pad 1: (no net) -> col7_rh
- SW_RH_07 pad 2: (no net) -> Net-(D_RH_07-A)
- SW_RH_08 pad 1: (no net) -> col8_rh
- SW_RH_08 pad 2: (no net) -> Net-(D_RH_08-A)
- SW_RH_10 pad 1: (no net) -> col0_rh
- SW_RH_10 pad 2: (no net) -> Net-(D_RH_10-A)
- SW_RH_11 pad 1: (no net) -> SW_RH_41_A
- SW_RH_11 pad 2: (no net) -> Net-(D_RH_11-A)
- SW_RH_12 pad 1: (no net) -> col2_rh
- SW_RH_12 pad 2: (no net) -> Net-(D_RH_12-A)
- SW_RH_13 pad 1: (no net) -> col3_rh
- SW_RH_13 pad 2: (no net) -> Net-(D_RH_13-A)
- SW_RH_14 pad 1: (no net) -> col4_rh
- SW_RH_14 pad 2: (no net) -> Net-(D_RH_14-A)
- SW_RH_15 pad 1: (no net) -> col5_rh
- SW_RH_15 pad 2: (no net) -> Net-(D_RH_15-A)
- SW_RH_16 pad 1: (no net) -> col6_rh
- SW_RH_16 pad 2: (no net) -> Net-(D_RH_16-A)
- SW_RH_17 pad 1: (no net) -> col7_rh
- SW_RH_17 pad 2: (no net) -> Net-(D_RH_17-A)
- SW_RH_18 pad 1: (no net) -> col8_rh
- SW_RH_18 pad 2: (no net) -> Net-(D_RH_18-A)
- SW_RH_20 pad 1: (no net) -> col0_rh
- SW_RH_20 pad 2: (no net) -> Net-(D_RH_20-A)
- SW_RH_21 pad 1: (no net) -> SW_RH_41_A
- SW_RH_21 pad 2: (no net) -> Net-(D_RH_21-A)
- SW_RH_22 pad 1: (no net) -> col2_rh
- SW_RH_22 pad 2: (no net) -> Net-(D_RH_22-A)
- SW_RH_23 pad 1: (no net) -> col3_rh
- SW_RH_23 pad 2: (no net) -> Net-(D_RH_23-A)
- SW_RH_24 pad 1: (no net) -> col4_rh
- SW_RH_24 pad 2: (no net) -> Net-(D_RH_24-A)
- SW_RH_25 pad 1: (no net) -> col5_rh
- SW_RH_25 pad 2: (no net) -> Net-(D_RH_25-A)
- SW_RH_26 pad 1: (no net) -> col6_rh
- SW_RH_26 pad 2: (no net) -> Net-(D_RH_26-A)
- SW_RH_27 pad 1: (no net) -> col7_rh
- SW_RH_27 pad 2: (no net) -> Net-(D_RH_27-A)
- SW_RH_28 pad 1: (no net) -> col8_rh
- SW_RH_28 pad 2: (no net) -> Net-(D_RH_28-A)
- SW_RH_30 pad 1: (no net) -> col0_rh
- SW_RH_30 pad 2: (no net) -> Net-(D_RH_30-A)
- SW_RH_31 pad 1: (no net) -> SW_RH_41_A
- SW_RH_31 pad 2: (no net) -> Net-(D_RH_31-A)
- SW_RH_32 pad 1: (no net) -> col2_rh
- SW_RH_32 pad 2: (no net) -> Net-(D_RH_32-A)
- SW_RH_33 pad 1: (no net) -> col3_rh
- SW_RH_33 pad 2: (no net) -> Net-(D_RH_33-A)
- SW_RH_34 pad 1: (no net) -> col4_rh
- SW_RH_34 pad 2: (no net) -> Net-(D_RH_34-A)
- SW_RH_35 pad 1: (no net) -> col5_rh
- SW_RH_35 pad 2: (no net) -> Net-(D_RH_35-A)
- SW_RH_36 pad 1: (no net) -> col6_rh
- SW_RH_36 pad 2: (no net) -> Net-(D_RH_36-A)
- SW_RH_37 pad 1: (no net) -> col7_rh
- SW_RH_37 pad 2: (no net) -> Net-(D_RH_37-A)
- SW_RH_38 pad 1: (no net) -> col8_rh
- SW_RH_38 pad 2: (no net) -> Net-(D_RH_38-A)
- SW_RH_40 pad 1: (no net) -> col0_rh
- SW_RH_40 pad 2: (no net) -> Net-(D_RH_40-A)
- SW_RH_42 pad 1: (no net) -> col2_rh
- SW_RH_42 pad 2: (no net) -> Net-(D_RH_42-A)
- SW_RH_43 pad 1: (no net) -> col3_rh
- SW_RH_43 pad 2: (no net) -> Net-(D_RH_43-A)
- SW_RH_44 pad 1: (no net) -> col4_rh
- SW_RH_44 pad 2: (no net) -> Net-(D_RH_44-A)
- SW_RH_45 pad 1: (no net) -> col5_rh
- SW_RH_45 pad 2: (no net) -> Net-(D_RH_45-A)
- SW_RH_46 pad 1: (no net) -> col6_rh
- SW_RH_46 pad 2: (no net) -> Net-(D_RH_46-A)
- SW_RH_47 pad 1: (no net) -> col7_rh
- SW_RH_47 pad 2: (no net) -> Net-(D_RH_47-A)
- SW_RH_48 pad 1: (no net) -> col8_rh
- SW_RH_48 pad 2: (no net) -> Net-(D_RH_48-A)
- SW_RH_50 pad 1: (no net) -> col0_rh
- SW_RH_50 pad 2: (no net) -> Net-(D_RH_50-A)
- SW_RH_51 pad 1: (no net) -> SW_RH_41_A
- SW_RH_51 pad 2: (no net) -> Net-(D_RH_51-A)
- SW_RH_52 pad 1: (no net) -> col2_rh
- SW_RH_52 pad 2: (no net) -> Net-(D_RH_52-A)
- SW_RH_53 pad 1: (no net) -> col3_rh
- SW_RH_53 pad 2: (no net) -> Net-(D_RH_53-A)
- SW_RH_54 pad 1: (no net) -> col4_rh
- SW_RH_54 pad 2: (no net) -> Net-(D_RH_54-A)
- SW_RH_55 pad 1: (no net) -> col5_rh
- SW_RH_55 pad 2: (no net) -> Net-(D_RH_55-A)
- SW_RH_56 pad 1: (no net) -> col6_rh
- SW_RH_56 pad 2: (no net) -> Net-(D_RH_56-A)
- SW_RH_57 pad 1: (no net) -> col7_rh
- SW_RH_57 pad 2: (no net) -> Net-(D_RH_57-A)
- SW_RH_58 pad 1: (no net) -> col8_rh
- SW_RH_58 pad 2: (no net) -> Net-(D_RH_58-A)
Other:
- board size 216.5 x 156.6 mm -> 15 x 15 mm
- board text added: "locked"
- board text removed: "1.75u"
- board text removed: "2.25u"

Commit message: pico diode placement
Parts:
- SWLH_ROT1, SWRH_ROT1: moved to F.Cu
- moved D_LH_58 261.0 mm to (-242.1, 1.23)
- moved D_RH_38 248.5 mm to (173.0, -58.3)
- moved D_LH_57 243.7 mm to (-218.3, 1.23)
- moved D_RH_47 235.5 mm to (146.8, -20.2)
- moved D_LH_37 226.8 mm to (-223.0, -36.9)
- moved D_LH_56 225.6 mm to (-196.8, -4.28)
- moved D_LH_27 224.4 mm to (-220.7, -55.9)
- moved D_RH_08 217.7 mm to (177.8, -77.1)
- moved D_LH_07 212.6 mm to (-223.9, -113.0)
- moved D_LH_55 209.8 mm to (-177.8, -9.78)
- moved D_LH_17 209.3 mm to (-215.9, -75.0)
- moved D_RH_18 208.0 mm to (149.2, -77.4)
- moved D_RH_28 207.4 mm to (149.2, -58.3)
- moved D_LH_53 207.2 mm to (-144.1, 8.83), turned to 172 degrees
- moved D_RH_46 204.6 mm to (111.1, -25.7)
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
Commit message: Spun out double-sided into corner-oled variant
Parts:
- moved L_RH_47 296.4 mm to (146.8, -34.1)
- moved L_RH_48 291.9 mm to (161.1, -53.1)
- moved L_RH_58 281.4 mm to (156.4, -15.0)
- moved L_LH_47 279.0 mm to (-227.8, -31.7)
- moved L_RH_38 272.6 mm to (173.0, -72.2)
- moved L_RH_46 270.9 mm to (111.1, -39.6)
- moved L_LH_58 267.9 mm to (-242.1, -12.7)
- moved L_RH_57 265.7 mm to (132.6, -15.0)
- moved L_RH_8 255.5 mm to (177.8, -91.2)
- moved L_LH_57 254.3 mm to (-218.3, -12.7)
- moved L_RH_37 250.7 mm to (130.2, -53.1)
- moved L_RH_18 249.6 mm to (149.2, -91.2)
- moved L_RH_56 249.5 mm to (111.1, -20.5)
- moved L_LH_37 249.4 mm to (-223.0, -50.8)
- moved L_LH_50 247.4 mm to (-91.5, 9.61), turned to -98 degrees
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
Commit message: Added 'simple' variant
Parts:
- added D1: D, ergodonk_pico:D3_TH_SMD_v2, F.Cu at (106.6, -161.0)
- added J1: AudioJack4, ergodonk_kicad_library:MJ-4PP-9_CANTOR_KITCHEN_SINK, F.Cu at (89.8, -161.4)
- added J4: AudioJack4, ergodonk_kicad_library:MJ-4PP-9_CANTOR_KITCHEN_SINK, F.Cu at (98.7, -161.4)
- added U2: Pico, ergodonk_pico:RPi_Pico_SMD_TH_DS_Ergodonk_v1, B.Cu at (35.7, -109.4)
- moved OL1 375.6 mm to (98.6, -176.6)
- moved Q1 249.4 mm to (-233.6, -98.8), turned to -90 degrees
- moved LS1 245.6 mm to (-214.2, -102.8), turned to 90 degrees
- moved S1 237.1 mm to (-197.7, -106.2)
- renumbered U2 to U1
Connections:
- SWRH_ROT1 pad A: encA -> encA_rh
- SWRH_ROT1 pad B: encB -> encB_rh
- U1 pad 20: col7 -> LED
- U1 pad 24: col8 -> unconnected-(U1-GPIO18-Pad24)
- U1 pad 25: LED -> unconnected-(U1-GPIO19-Pad25)
- U1 pad 26: SDA -> SOLENOID_CONTROL
- U1 pad 27: SCL -> SPEAKER
- U1 pad 29: SOLENOID_CONTROL -> col8
- U1 pad 31: SPEAKER -> SDA
- U1 pad 32: unconnected-(U2-GPIO27_ADC1-Pad32) -> SCL
- U1 pad 34: unconnected-(U2-GPIO28_ADC2-Pad34) -> col7

Commit message: Checkpoint commit
Parts:
- added ?: , clipboard:39367019-bb4e-49d1-b84f-72ef74cff27d, F.Cu at (-139.3, -159.9)
- added ?: , clipboard:39367019-bb4e-49d1-b84f-72ef74cff27d, F.Cu at (-227.3, -96.6)
- added ?: , clipboard:39367019-bb4e-49d1-b84f-72ef74cff27d, F.Cu at (147.4, -116.8)
- added ?: , clipboard:39367019-bb4e-49d1-b84f-72ef74cff27d, F.Cu at (-65.2, -153.0)
- added ?: , clipboard:39367019-bb4e-49d1-b84f-72ef74cff27d, F.Cu at (-14.7, -122.2)
- added OL1: OLED, ergodonk_kicad_library:OLED SSD1306 128x64 UNVERIFIED, F.Cu at (-130.4, -157.7)
- moved J1 175.7 mm to (-78.9, -112.0), turned to -56.3 degrees
- moved OL1 157.0 mm to (-56.2, -150.8)
- moved J4 126.8 mm to (-15.4, -106.1), turned to 90 degrees
