File: ergodonk_simple/ergodonk_simple.kicad_sch (KiCad schematic)
At the start: 130 parts, among them J10 Pimaroni Trackball, J2 4PIN, Q1 TIP120, SW0 SW_PUSH_LED, SW08_RH10 SW_PUSH_LED, SW1 SW_PUSH_LED, SW10 SW_PUSH_LED, SW11 SW_PUSH_LED, SW12 SW_PUSH_LED, SW13 SW_PUSH_LED, SW14 SW_PUSH_LED, SW15 SW_PUSH_LED, SW16 SW_PUSH_LED, SW17 SW_PUSH_LED, SW18_RH10 SW_PUSH_LED, SW2 SW_PUSH_LED, SW20 SW_PUSH_LED, SW21 SW_PUSH_LED, SW22 SW_PUSH_LED, SW23 SW_PUSH_LED, SW24 SW_PUSH_LED, SW25 SW_PUSH_LED, SW26 SW_PUSH_LED, SW27 SW_PUSH_LED, SW28_RH10 SW_PUSH_LED, SW3 SW_PUSH_LED, SW30 SW_PUSH_LED, SW31 SW_PUSH_LED, SW32 SW_PUSH_LED, SW33 SW_PUSH_LED, SW34 SW_PUSH_LED, SW35 SW_PUSH_LED, SW36 SW_PUSH_LED, SW37 SW_PUSH_LED, SW38_RH10 SW_PUSH_LED, SW4 SW_PUSH_LED, SW40 SW_PUSH_LED, SW42 SW_PUSH_LED, SW43 SW_PUSH_LED, SW44 SW_PUSH_LED, SW45 SW_PUSH_LED, SW46 SW_PUSH_LED, SW47 SW_PUSH_LED, SW48_RH10 SW_PUSH_LED, SW5 SW_PUSH_LED, SW50 SW_PUSH_LED, SW51 SW_PUSH_LED, SW52 SW_PUSH_LED, SW53 SW_PUSH_LED, SW54 SW_PUSH_LED, SW55 SW_PUSH_LED, SW56 SW_PUSH_LED, SW57 SW_PUSH_LED, SW58 SW_PUSH_LED, SW6 SW_PUSH_LED, SW7 SW_PUSH_LED, U11 Pico

Commit message: simple variant routing checkpoint commit
Parts:
- U11: footprint ergodonk_pico:RPi_Pico_SMD_TH_DS_Ergodonk_v1 -> ergodonk_simple:RPi_Pico_SMD_TH_DS_Simple_v1
Connections:
- net GND: now also U11.13 (GND), U11.18 (GND), U11.3 (GND), U11.8 (GND)
- net SCL: no longer U11.32 (GPIO27_ADC1)
- net SDA: no longer U11.31 (GPIO26_ADC0)
- net SOLENOID_CONTROL: now also U11.22 (GPIO17); no longer U11.26 (GPIO20)
- net SW41A: now also U11.16 (GPIO12); no longer U11.14 (GPIO10)
- net col0: now also U11.15 (GPIO11); no longer U11.12 (GPIO9)
- net col2: now also U11.4 (GPIO2); no longer U11.15 (GPIO11)
- net col3: now also U11.26 (GPIO20); no longer U11.16 (GPIO12)
- net col4: now also U11.27 (GPIO21); no longer U11.17 (GPIO13)
- net col5: now also U11.29 (GPIO22); no longer U11.19 (GPIO14)
- net col6: now also U11.31 (GPIO26_ADC0); no longer U11.4 (GPIO2)
- net col7: now also U11.32 (GPIO27_ADC1); no longer U11.5 (GPIO3)
- net col8: now also U11.34 (GPIO28_ADC2); no longer U11.20 (GPIO15)
- net encA: now also U11.12 (GPIO9); no longer U11.25 (GPIO19)
- net encB: now also U11.14 (GPIO10); no longer U11.24 (GPIO18)
- net row2: now also U11.11 (GPIO8); no longer U11.6 (GPIO4)
- net row3: now also U11.17 (GPIO13); no longer U11.9 (GPIO6)
- net row4: now also U11.19 (GPIO14); no longer U11.10 (GPIO7)
- net row5: now also U11.20 (GPIO15); no longer U11.11 (GPIO8)
- no-connect marks 16 -> 13

Commit message: CHeckpoint commit before simple MCU move
Parts:
- H1, H10, H11, H12, H13, H2, H3, H4, H5, H6, H7, H8, H9: footprint MountingHole:MountingHole_2.2mm_M2_Pad_Via -> ergodonk_simple:Hole from sofle for M2 posts gold rimmer
- J10: footprint ergodonk_kicad_library:pimoroni_trackball -> ergodonk_simple:pimoroni_trackball_no_cutout
- Q1: footprint ergodonk_kicad_library:Tip 120 with heatsink -> ergodonk_simple:TO-220-3_Horizontal_TabDown
Connections:
- net GND: now also J2.1; no longer J2.2
- net SCL: now also U11.10 (GPIO7)
- net SDA: now also U11.9 (GPIO6)
- net SOLENOID_CONTROL: now also U11.25 (GPIO19); no longer U11.22 (GPIO17)
- net VCC: now also J2.2; no longer J2.1
- net RX: now reaches U11.2 (GPIO1)
- net RX: now also J2.3
- net TX: now reaches J2.4
- net TX: now also U11.1 (GPIO0)
- removed net DATA: J2.3, U11.1 (GPIO0)
- no-connect marks 13 -> 11

Commit message: pcb simple with encoder checkpoint before outline mod
Parts:
- added J12: Conn_01x08_Socket, Connector_PinHeader_2.54mm:PinHeader_1x08_P2.54mm_Vertical, symbol Connector:Conn_01x08_Socket
- added SW18: RotaryEncoder, ergodonk_simple:Bourns Hollow Encoder V1, symbol Device:RotaryEncoder
Connections:
- net GND: now also J12.2 (Pin_2), SW18.C
- net SCL: now also U11.22 (GPIO17); no longer U11.10 (GPIO7)
- net SDA: now also U11.21 (GPIO16); no longer U11.9 (GPIO6)
- net SOLENOID_CONTROL: now also U11.10 (GPIO7); no longer U11.25 (GPIO19)
- net SW41A: now also U11.4 (GPIO2); no longer U11.16 (GPIO12)
- net col0: now also U11.11 (GPIO8); no longer U11.15 (GPIO11)
- net col2: now also U11.5 (GPIO3); no longer U11.4 (GPIO2)
- net col3: now also U11.6 (GPIO4); no longer U11.26 (GPIO20)
- net col4: now also U11.7 (GPIO5); no longer U11.27 (GPIO21)
- net col5: now also U11.34 (GPIO28_ADC2); no longer U11.29 (GPIO22)
- net col6: now also U11.32 (GPIO27_ADC1); no longer U11.31 (GPIO26_ADC0)
- net col7: now also U11.31 (GPIO26_ADC0); no longer U11.32 (GPIO27_ADC1)
- net col8: now also U11.29 (GPIO22); no longer U11.34 (GPIO28_ADC2)
- net encA: now also U11.20 (GPIO15), SW18.A; no longer U11.12 (GPIO9)
- net encB: now also U11.19 (GPIO14), SW18.B; no longer U11.14 (GPIO10)
- net row0: now also U11.9 (GPIO6); no longer U11.7 (GPIO5)
- net row1: now also U11.17 (GPIO13); no longer U11.21 (GPIO16)
- net row2: now also U11.16 (GPIO12); no longer U11.11 (GPIO8)
- net row3: now also U11.14 (GPIO10); no longer U11.17 (GPIO13)
- net row4: now also U11.15 (GPIO11); no longer U11.19 (GPIO14)
- net row5: now also U11.12 (GPIO9); no longer U11.20 (GPIO15)
- net SC: now reaches U11.24 (GPIO18)
- net SC: now also J12.5 (Pin_5)
- net VI: now reaches U11.36 (3V3)
- net VI: now also J12.8 (Pin_8)
- new net MI: J12.7 (Pin_7), U11.26 (GPIO20)
- new net MO: J12.6 (Pin_6), U11.25 (GPIO19)
- new net SS: J12.4 (Pin_4), U11.27 (GPIO21)
- no-connect marks 11 -> 12
Other:
- note added: "Hollow Rotary Encoder for trackball"

Commit message: Flipped rotary encoder to backside
Parts:
- SW0, SW1, SW10, SW11, SW12, SW13, SW14, SW15, SW16, SW17, SW2, SW20, SW21, SW22, SW23, SW24, SW25, SW26, SW3, SW30, SW31, SW32, SW33, SW34, SW35, SW36, SW4, SW40, SW42, SW43, SW44, SW45, SW46, SW5, SW50, SW51, SW52, SW53, SW54, SW55, SW56, SW57, SW58, SW6, SW7: footprint ergodonk_pico:Cherry_MX_DS_Hotswap_1U_sofle3b v2 -> ergodonk_simple:Cherry_MX_DS_Hotswap_1U_sofle3b v3

Commit message: SENT OUT FOR PRODUCTION
Parts:
- added H14, H15, H16, H17, H18, H19, H20, H21, H22, H23, H24, H25: MountingHole, ergodonk_simple:M2_Hole_fancy_for_bolt-on-plate, symbol Mechanical:MountingHole
- D_SOL_1: footprint ergodonk_kicad_library:MUR340S_IN4001_TH_HYBRID -> ergodonk_simple:MUR340S_IN4001_TH_HYBRID
- H11, H12, H13: footprint ergodonk_simple:Hole from sofle for M2 posts gold rimmer -> ergodonk_simple:M2_Hole_fancy_for_bolt-on-plate
- J10: footprint ergodonk_simple:pimoroni_trackball_no_cutout -> ergodonk_simple:Pimaroni_PinHeader_1x05_P2.54mm_Vertical Sofle v3b
- SW18: footprint ergodonk_simple:Bourns Hollow Encoder V1 -> ergodonk_simple:Bourns Hollow Encoder high plate_donk_holes
- SWLH_ROT1: footprint ergodonk_kicad_library:RotaryEncoder_EC11_ergodonk_variant -> ergodonk_simple:RotaryEncoder_EC11_ergodonk_variant
Other:
- note added: "TRRS jack. Serial config is default Jumper must be soldered for TX/RX"
- note removed: "TRRS jack. (Serial config is default)"
- moved on the sheet: D49, H11, H12, H13, S1, U11

Commit message: Added underglow to schematic
Parts:
- added JP1: Level shifter bypass jumper, sofle_v3b:Level Shifter Bypass Jumper, symbol Jumper:SolderJumper_2_Open
- added JP10: SolderJumper_3_Open, symbol Jumper:SolderJumper_3_Open
- added unit 2 of SW1 (x7)
- added U2: SN74AHCT1G125, sofle_v3b:SN74AHCT1G125 - Junco, symbol Junco:SN74AHCT1G125
Connections:
- net GND: now also SW1.3 (GND), SW1.3 (GND), SW1.3 (GND), SW1.3 (GND), SW1.3 (GND), SW1.3 (GND), SW1.3 (GND), U2.1 (OE), U2.3 (GND)
- net RX: now also JP10.3 (B); no longer U11.2 (GPIO1)
- net VCC: now also U2.5 (VCC)
- new net: SW1.2 (DOUT), SW1.4 (DIN) (x6)
- new net: JP10.2 (C), U11.2 (GPIO1)
- new net: JP1.2 (B), SW1.4 (DIN), U2.4 (DOUT)
- new net LED: JP1.1 (A), JP10.1 (A), U2.2 (DIN)
- new net VDD: SW1.1 (VDD), SW1.1 (VDD), SW1.1 (VDD), SW1.1 (VDD), SW1.1 (VDD), SW1.1 (VDD), SW1.1 (VDD)
Other:
- note added: "LED Level shifter"
