File: ergodonk_pico_zero/ergodonk_pico_zero.kicad_pcb (KiCad board)
At the start: 2 copper layers, 15 x 15 mm, 340 parts, among them J1 AudioJack4, J2 Pimaroni Trackball, J3 AudioJack4, J4 AudioJack4, Q1 TIP120, U1 Pico, U2 Pico

Commit message: Basic routing on ergodonk pico zero simple
Parts:
- removed ?: , clipboard:39367019-bb4e-49d1-b84f-72ef74cff27d
- removed J2: Pimaroni Trackball, ergodonk_kicad_library:pimoroni_trackball
- removed L_LH_00, L_LH_1, L_LH_10, L_LH_11, L_LH_12, L_LH_13, L_LH_14, L_LH_15, L_LH_16, L_LH_17, L_LH_2, L_LH_20, L_LH_21, L_LH_22, L_LH_23, L_LH_24, L_LH_25, L_LH_26, L_LH_27, L_LH_3, L_LH_30, L_LH_31, L_LH_32, L_LH_33, L_LH_34, L_LH_35, L_LH_36, L_LH_37, L_LH_4, L_LH_40, L_LH_41, L_LH_42, L_LH_43, L_LH_44, L_LH_45, L_LH_46, L_LH_47, L_LH_5, L_LH_50, L_LH_51, L_LH_52, L_LH_53, L_LH_54, L_LH_55, L_LH_56, L_LH_57, L_LH_58, L_LH_6, L_LH_7, L_RH_00, L_RH_1, L_RH_10, L_RH_11, L_RH_12, L_RH_13, L_RH_14, L_RH_15, L_RH_16, L_RH_17, L_RH_18, L_RH_2, L_RH_20, L_RH_21, L_RH_22, L_RH_23, L_RH_24, L_RH_25, L_RH_26, L_RH_27, L_RH_28, L_RH_3, L_RH_30, L_RH_31, L_RH_32, L_RH_33, L_RH_34, L_RH_35, L_RH_36, L_RH_37, L_RH_38, L_RH_4, L_RH_40, L_RH_41, L_RH_42, L_RH_43, L_RH_44, L_RH_45, L_RH_46, L_RH_47, L_RH_48, L_RH_5, L_RH_50, L_RH_51, L_RH_52, L_RH_53, L_RH_54, L_RH_55, L_RH_56, L_RH_57, L_RH_58, L_RH_6, L_RH_7, L_RH_8: SK6812MINI-E, ergodonk_pico:SK6812-MINI-E
- removed OL1: OLED, ergodonk_kicad_library:OLED SSD1306 128x64 UNVERIFIED
- removed U1, U2: Pico, ergodonk_pico:RPi_Pico_SMD_TH_DS_Ergodonk_v1
- added MCU1: rp2040-zero, ergodonk_kicad_library:rp2040 Zero DS, F.Cu at (-243.0, -119.7)
- added MCU2: rp2040-zero, ergodonk_kicad_library:rp2040 Zero DS, F.Cu at (154.6, -122.4)
- moved Q1 116.7 mm to (-171.8, 0.21)
- moved D_RH_10 2.75 mm to (-6.17, -66.1)
- moved D_RH_21 2.75 mm to (15.9, -66.1)
- moved D_RH_00 2.75 mm to (-6.17, -85.1)
- moved D_RH_11 2.75 mm to (15.9, -85.1)
- moved D_RH_20 2.75 mm to (-6.17, -47.0)
- moved D_RH_31 2.75 mm to (15.9, -47.0)
- moved D_RH_41 2.75 mm to (15.9, -27.9)
- moved SWRH_ROT1 2.75 mm to (15.9, -36.9)
- moved SW_RH_00 2.75 mm to (-6.17, -94.0)
- moved SW_RH_10 2.75 mm to (-6.17, -75.0)
- moved SW_RH_11 2.75 mm to (15.9, -94.0)
- moved SW_RH_20 2.75 mm to (-6.17, -55.9)
- moved SW_RH_21 2.75 mm to (15.9, -75.0)
- moved SW_RH_31 2.75 mm to (15.9, -55.9)
Other:
- board size 15 x 15 mm -> 9.3 x 11.3 mm
