File: ergodonk_pico_zero/ergodonk_pico_zero.kicad_sch (KiCad schematic)
At the start: 339 parts, among them J1 AudioJack4, J2 Conn_01x08_Socket, J4 AudioJack4, Q1 TIP120, U1 Pico, U2 Pico

Commit message: Basic routing on ergodonk pico zero simple
Parts:
- removed D1, D102: D, ergodonk_pico:D3_TH_SMD_v2, symbol Device:D
- removed J2: Conn_01x08_Socket, symbol Connector:Conn_01x08_Socket
- removed LS1: AST1109MLTRQ_MAL, ergodonk_kicad_library:AST1109MLTRQ, symbol AST1109MLTRQ:AST1109MLTRQ
- removed L_LH_00, L_LH_1, L_LH_10, L_LH_11, L_LH_12, L_LH_13, L_LH_14, L_LH_15, L_LH_16, L_LH_17, L_LH_2, L_LH_20, L_LH_21, L_LH_22, L_LH_23, L_LH_24, L_LH_25, L_LH_26, L_LH_27, L_LH_3, L_LH_30, L_LH_31, L_LH_32, L_LH_33, L_LH_34, L_LH_35, L_LH_36, L_LH_37, L_LH_4, L_LH_40, L_LH_41, L_LH_42, L_LH_43, L_LH_44, L_LH_45, L_LH_46, L_LH_47, L_LH_5, L_LH_50, L_LH_51, L_LH_52, L_LH_53, L_LH_54, L_LH_55, L_LH_56, L_LH_57, L_LH_58, L_LH_6, L_LH_7, L_RH_00, L_RH_1, L_RH_10, L_RH_11, L_RH_12, L_RH_13, L_RH_14, L_RH_15, L_RH_16, L_RH_17, L_RH_18, L_RH_2, L_RH_20, L_RH_21, L_RH_22, L_RH_23, L_RH_24, L_RH_25, L_RH_26, L_RH_27, L_RH_28, L_RH_3, L_RH_30, L_RH_31, L_RH_32, L_RH_33, L_RH_34, L_RH_35, L_RH_36, L_RH_37, L_RH_38, L_RH_4, L_RH_40, L_RH_41, L_RH_42, L_RH_43, L_RH_44, L_RH_45, L_RH_46, L_RH_47, L_RH_48, L_RH_5, L_RH_50, L_RH_51, L_RH_52, L_RH_53, L_RH_54, L_RH_55, L_RH_56, L_RH_57, L_RH_58, L_RH_6, L_RH_7, L_RH_8: SK6812MINI-E, ergodonk_pico:SK6812-MINI-E, symbol Ergodonk_symbols:SK6812MINI
- removed OL1: OLED, ergodonk_kicad_library:OLED SSD1306 128x64 UNVERIFIED, symbol kbd:OLED
- removed U1, U2: Pico, ergodonk_pico:RPi_Pico_SMD_TH_DS_Ergodonk_v1, symbol Pico:Pico
- added MCU1: rp2040-zero, ergodonk_kicad_library:rp2040 Zero DS, symbol zzkeeb:MCU_rp2040-zero
- MCU1: footprint zzkeeb:MCU_rp2040-zero-tht-pads -> ergodonk_kicad_library:rp2040 Zero DS
Connections:
- net +5V: now also MCU1.23 (5V)
- net GND: now also MCU1.22 (GND)
- net LED: now also MCU1.20 (29); no longer MCU1.20 (29)
- net SOLENOID_CONTROL: now also MCU1.20 (29)
- net SW_RH_41_A: now also MCU1.4 (3)
- net VCC: now also MCU1.21 (3V3)
- net col0_rh: now also MCU1.3 (2)
- net col2_rh: now also MCU1.5 (4)
- net col3_rh: now also MCU1.6 (5)
- net col4_rh: now also MCU1.7 (6)
- net col5_rh: now also MCU1.8 (7)
- net col6_rh: now also MCU1.9 (8)
- net col7_rh: now also MCU1.13 (12)
- net col8_rh: now also MCU1.12 (11)
- net data1RX: now also MCU1.2 (1)
- net data1TX: now also MCU1.1 (0)
- net encA_rh: now also MCU1.11 (10)
- net encB_rh: now also MCU1.10 (9)
- net row0_rh: now also MCU1.19 (28)
- net row1_rh: now also MCU1.18 (27)
- net row2_rh: now also MCU1.17 (26)
- net row3_rh: now also MCU1.16 (15)
- net row4_rh: now also MCU1.15 (14)
- net row5_rh: now also MCU1.14 (13)
- no-connect marks 20 -> 2
Other:
- note removed: "OLED (Chain to pimaroni for sharing bus?)"
- note removed: "PMW3360 Trackball https://wylderbuilds.com/trackball-install"
- note removed: "Speaker"
